File: super-met/super-met.kicad_sch (KiCad schematic)
At the start: 60 parts, among them J1 Power conn, J2 Conn_01x08, J3 Conn_01x08, J4 Conn_01x08, J5 Conn_01x08, J6 Частицы_power, J7 Частицы_uart, Q1 AO3400A, Q10 AO3400A, Q11 AO3400A, Q12 AO3400A, Q2 AO3400A, Q3 AO3400A, Q4 AO3400A, Q5 AO3400A, Q6 AO3400A, Q7 AO3400A, Q8 AO3400A, Q9 AO3400A, U10 74HC595, U11 74HC595, U4 74HC4052D, U5 ADS1115IDGS, U6 ADS1115IDGS, U7 ADS1115IDGS, U8 ADS1115IDGS, U9 ESP-01v090

Commit message: adding v6 (libst included and ported))
Parts:
- removed RN3, RN4: 4.7K, Resistor_SMD:R_Array_Convex_4x0603, symbol Device:R_Pack04
- added J10, J11, J8, J9: Conn_01x08, Connector_JST:JST_PH_S8B-PH-K_1x08_P2.00mm_Horizontal, symbol Connector_Generic:Conn_01x08
- renumbered RN5 to RN3, RN6 to RN4, RN7 to RN5, U9 to U10, U10 to U11, 12 to U12, U11 to U13, 13 to U14, 11 to U4, U4 to U5, U5 to U6, U6 to U7, U7 to U8, U8 to U9
Connections:
- net 3.3v: now also RN1.1 (R1.1), RN1.2 (R2.1); no longer RN1.3 (R3.1), RN1.4 (R4.1)
- net 5.2v: now also RN1.3 (R3.1), RN1.4 (R4.1); no longer RN1.1 (R1.1), RN1.2 (R2.1)
- net s0: now also Q12.3 (D), RN5.8 (R1.2); no longer Q12.2 (S), RN5.5 (R4.2)
- net s1: now also Q11.3 (D), RN5.7 (R2.2); no longer Q11.2 (S), RN5.6 (R3.2)
- net sim800_rx: now also RN1.5 (R4.2); no longer RN1.7 (R2.2)
- net sim800_tx: now also RN1.6 (R3.2); no longer RN1.8 (R1.2)
- net uart_mux_rx: now also Q6.2 (S), RN2.6 (R3.2); no longer Q6.3 (D), RN2.8 (R1.2)
- net uart_mux_tx: now also Q5.2 (S), RN2.5 (R4.2); no longer Q5.3 (D), RN2.7 (R2.2)
- net at Q3.2 (S), U4.4 (Rx): now also RN1.7 (R2.2); no longer RN1.6 (R3.2)
- net at Q4.2 (S), U4.5 (Tx): now also RN1.8 (R1.2); no longer RN1.5 (R4.2)
- new net: Q12.2 (S), RN5.5 (R4.2), U12.25 (PA0)
- new net: Q11.2 (S), RN5.6 (R3.2), U12.26 (PA1)
- new net: Q5.3 (D), RN2.7 (R2.2), U5.13 (1Z)
- new net: Q6.3 (D), RN2.8 (R1.2), U5.3 (2Z)
- no-connect marks 54 -> 46
Other:
- added sheet Sensors (sensors.kicad_sch)
- note added: "en на каждый датчик и 16 каналов датчиков пока избыточно + цифровые датчики также будут на этой плате, поэтому потом сюда выведется i2c + пины управления"
- note added: "тут будет 2я плата с сенсорами"
- moved on the sheet: C1, J1, J4, J5, Q1, Q11, Q12, Q2, Q3, Q4, R1, R2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
