File: super-met v6/super-met-v6/sensors.kicad_sch (KiCad schematic)
At the start: 0 parts

Commit message: sensors board
Parts:
- added C1: 10uF, Capacitor_SMD:C_1206_3216Metric, symbol Device:C_Small
- added J1, J2, J3: Conn_01x08, Connector_JST:JST_PH_S8B-PH-K_1x08_P2.00mm_Horizontal, symbol Connector_Generic:Conn_01x08
- added J4, J5: Conn_01x04, Connector_PinHeader_2.54mm:PinHeader_1x04_P2.54mm_Horizontal, symbol Connector_Generic:Conn_01x04
- added Q1, Q10, Q11, Q12, Q2, Q3, Q4, Q5, Q6, Q7, Q8, Q9: AO3400A, Package_TO_SOT_SMD:SOT-23, symbol Transistor_FET:AO3400A
- added R1, R13, R14, R15, R19, R2, R21, R22, R3, R7, R8, R9: 100, Resistor_SMD:R_0805_2012Metric_Pad1.20x1.40mm_HandSolder, symbol Device:R_Small
- added R10, R11, R12, R16, R17, R18, R20, R23, R24, R4, R5, R6: 1k, Resistor_SMD:R_0805_2012Metric_Pad1.20x1.40mm_HandSolder, symbol Device:R_Small
- added U1, U11, U12, U2, U3, U4, U5, U6, U7, U8: MQ GENERIC BOARD SENSOR, super-met:MQ BLUE GENERIC MODULE, symbol super-met:MQ GENERIC BOARD SENSOR
- added U10: MS-1100, super-met:MS-1100, symbol super-met:MS-1100
- added U13: CCS811, super-met:CCS811, symbol super-met:CCS811
- added U14: AHT10 MODULE, super-met:AHT10 FOOT PRINT, symbol super-met:AHT10 MODULE
- added U9: MICS-6814, super-met:MICS-6814, symbol super-met:MICS-6814
Connections:
- new net: Q3.1 (G), R3.2, R6.1
- new net: Q10.3 (D), U10.4 (Gnd)
- new net: Q2.1 (G), R2.2, R5.1
- new net: Q12.1 (G), R22.2, R24.1
- new net: Q5.3 (D), U5.2 (Gnd)
- new net: Q4.1 (G), R10.1, R7.2
- new net: Q11.1 (G), R21.2, R23.1
- new net: Q6.3 (D), U6.2 (Gnd)
- new net: Q1.1 (G), R1.2, R4.1
- new net: Q9.1 (G), R15.2, R18.1
- new net: Q8.3 (D), U7.2 (Gnd)
- new net: Q9.3 (D), U8.2 (Gnd)
- new net: Q5.1 (G), R11.1, R8.2
- new net: Q4.3 (D), U4.2 (Gnd)
- new net: Q8.1 (G), R14.2, R17.1
- new net: Q7.1 (G), R13.2, R16.1
- new net: Q7.3 (D), U9.4 (Gnd)
- new net: Q3.3 (D), U3.2 (Gnd)
- new net: Q2.3 (D), U2.2 (Gnd)
- new net: Q1.3 (D), U1.2 (Gnd)
- new net: Q11.3 (D), U11.2 (Gnd)
- new net: Q12.3 (D), U12.2 (Gnd)
- new net: Q10.1 (G), R19.2, R20.1
- new net: Q6.1 (G), R12.1, R9.2
- new net 3.3V_sub: J5.1 (Pin_1), U13.1 (Vcc), U14.4 (Vin)
- new net 5.2V_IN_sub: C1.1, J3.7 (Pin_7), U1.1 (Vcc), U10.1 (Vin), U11.1 (Vcc), U12.1 (Vcc), U2.1 (Vcc), U3.1 (Vcc), U4.1 (Vcc), U5.1 (Vcc), U6.1 (Vcc), U7.1 (Vcc), U8.1 (Vcc), U9.5 (Vin)
- new net GND2: C1.2, J3.8 (Pin_8), J5.2 (Pin_2), Q1.2 (S), Q10.2 (S), Q11.2 (S), Q12.2 (S), Q2.2 (S), Q3.2 (S), Q4.2 (S), Q5.2 (S), Q6.2 (S), Q7.2 (S), Q8.2 (S), Q9.2 (S), R10.2, R11.2, R12.2, R16.2, R17.2, R18.2, R20.2, R23.2, R24.2, R4.2, R5.2, R6.2, U13.2 (Gnd), U14.3 (Gnd)
- new net S10_EN_sub: J3.3 (Pin_3), U6.4 (A0)
- new net S10_OUT_sub: J3.4 (Pin_4), R9.1
- new net S11_12_13_EN_sub: J4.4 (Pin_4), R13.1
- new net S11_OUT_sub: J4.1 (Pin_1), U9.1 (CO)
- new net S12_OUT_sub: J4.2 (Pin_2), U9.2 (NH3)
- new net S13_OUT_sub: J4.3 (Pin_3), U9.3 (NO2)
- new net S14_EN_sub: J3.1 (Pin_1), R19.1
- new net S14_OUT_sub: J3.2 (Pin_2), U10.2 (Signal)
- new net S1_EN_sub: J1.7 (Pin_7), R1.1
- new net S1_OUT_sub: J1.8 (Pin_8), U1.4 (A0)
- new net S2_EN_sub: J1.5 (Pin_5), R7.1
- new net S2_OUT_sub: J1.6 (Pin_6), U4.4 (A0)
- new net S3_EN_sub: J1.3 (Pin_3), R14.1
- new net S3_OUT_sub: J1.4 (Pin_4), U7.4 (A0)
- new net S4_EN_sub: J1.1 (Pin_1), R21.1
- new net S4_OUT_sub: J1.2 (Pin_2), U11.4 (A0)
- new net S5_EN_sub: J2.7 (Pin_7), R2.1
- new net S5_OUT_sub: J2.8 (Pin_8), U2.4 (A0)
- new net S6_EN_sub: J2.5 (Pin_5), R8.1
- new net S6_OUT_sub: J2.6 (Pin_6), U5.4 (A0)
- new net S7_EN_sub: J2.3 (Pin_3), R15.1
- new net S7_OUT_sub: J2.4 (Pin_4), U8.4 (A0)
- new net S8_EN_sub: J2.1 (Pin_1), R22.1
- new net S8_OUT_sub: J2.2 (Pin_2), U12.4 (A0)
- new net S9_EN_sub: J3.5 (Pin_5), R3.1
- new net S9_OUT_sub: J3.6 (Pin_6), U3.4 (A0)
- new net SCL_sub: J5.4 (Pin_4), U13.3 (Scl), U14.2 (SCL)
- new net SDA_sub: J5.3 (Pin_3), U13.4 (Sda), U14.1 (SDA)
- no-connect marks 0 -> 15
Other:
- note added: "3.3v MAX"
- note added: "3.3v on I2c?"
