File: super-met v6/super-met-v6/super-met-v6.kicad_pcb (KiCad board)
At the start: 2 copper layers, 99.1 x 99.1 mm, 59 parts, among them J1 Conn_01x02, J2 Conn_01x08, J3 Conn_01x08, J4 Conn_01x04, J5 Conn_01x08, J6 Conn_01x04, J7 Conn_01x02, J8 Conn_01x02, Q1 AO3400A, Q10 AO3400A, Q11 AO3400A, Q12 AO3400A, Q2 AO3400A, Q3 AO3400A, Q4 AO3400A, Q5 AO3400A, Q6 AO3400A, Q7 AO3400A, Q8 AO3400A, Q9 AO3400A, U1 DC-DC_MOD, U10 74HC595, U11 GY-GPS6MV2, U12 ESP-01v090, U13 74HC4052D, U14 BLUEPILL, U2 DC-DC_MOD, U3 DC-DC_MOD, U4 ADS1115IDGS, U5 ADS1115IDGS, U6 ADS1115IDGS, U7 ADS1115IDGS, U8 74HC595, U9 SIM800L

Commit message: board in progress
Parts:
- added REF**: 0, Resistor_SMD:R_0603_1608Metric, B.Cu at (239.3, 75.7)
- added REF**: 0, Resistor_SMD:R_0603_1608Metric, B.Cu at (201.7, 81.8)
- added REF**: 0, Resistor_SMD:R_1206_3216Metric, B.Cu at (196.2, 68.4)
- added REF**: 0, Resistor_SMD:R_1206_3216Metric, B.Cu at (254.5, 82.3)
- C1, C2, C3, C4, C6, JP1, Q10, Q11, Q12, Q3, Q4, Q5, Q6, Q7, Q8, Q9, RN1, RN2, RN3, RN4, RN5, U10, U13, U4, U5, U6, U7, U8: moved to B.Cu
- moved TP1 152.6 mm to (231.1, 268.0)
- moved TP3 152.6 mm to (243.1, 260.0)
- moved TP4 152.6 mm to (236.1, 261.0)
- moved TP2 117.7 mm to (231.1, 257.8)
- moved C5 88.7 mm to (263.7, 95.0), turned to -90 degrees
- moved Q4 82.9 mm to (238.3, 69.1)
- moved RN1 80.1 mm to (230.6, 73.2)
- moved J7 71.1 mm to (152.4, 154.6), turned to 0 degrees
- moved TP5 71.0 mm to (151.1, 95.2)
- moved R4 64.5 mm to (138.8, 157.5), turned to -90 degrees
- moved Q1 64.4 mm to (142.2, 157.5)
- moved C1 61.8 mm to (275.0, 147.3), turned to 180 degrees
- moved C2 61.8 mm to (275.0, 139.3), turned to 180 degrees
- moved C3 61.8 mm to (275.0, 155.3), turned to 180 degrees
- moved C4 61.8 mm to (275.0, 143.3), turned to 180 degrees
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Connections:
- RN1 pad 2: 5.2v -> 3.3v
- RN1 pad 3: 3.3v -> 5.2v
- RN1 pad 6: /SCL1 -> Net-(Q4-Pad3)
- RN1 pad 7: Net-(Q4-Pad3) -> /SCL1
- RN2 pad 1: 5.2v -> 3.3v
- RN2 pad 4: 3.3v -> 5.2v
- RN2 pad 5: /SDA2 -> Net-(Q6-Pad3)
- RN2 pad 6: /SCL2 -> /SDA2
- RN2 pad 7: Net-(Q6-Pad3) -> Net-(Q5-Pad3)
- RN2 pad 8: Net-(Q5-Pad3) -> /SCL2
- RN3 pad 1: /sim800_tx -> Net-(Q8-Pad2)
- RN3 pad 2: /sim800_rx -> /sim800_tx
- RN3 pad 4: Net-(Q8-Pad2) -> /sim800_rx
- RN3 pad 5: 3.3v -> 5.2v
- RN3 pad 8: 5.2v -> 3.3v
- RN4 pad 1: /uart_mux_rx -> /uart_mux_tx
- RN4 pad 2: /uart_mux_tx -> Net-(Q9-Pad3)
- RN4 pad 3: Net-(Q9-Pad3) -> /uart_mux_rx
- RN4 pad 6: 5.2v -> 3.3v
- RN4 pad 7: 3.3v -> 5.2v
- RN5 pad 1: /uart_mux_s1 -> /uart_mux_s0
- RN5 pad 2: /uart_mux_s0 -> Net-(Q11-Pad3)
- RN5 pad 3: Net-(Q11-Pad3) -> /uart_mux_s1
- RN5 pad 6: 5.2v -> 3.3v
- RN5 pad 7: 3.3v -> 5.2v
- U10 pad 1: /s10_en_1 -> /s9_en_1
- U10 pad 15: /s9_en_1 -> /s11_12_13_en_1
- U10 pad 2: /s14_en_1 -> /s10_en_1
- U10 pad 3: /s11_12_13_en_1 -> /s14_en_1
- U13 pad 11: unconnected-(U13-Pad11) -> /gps_rx
- U13 pad 14: /gps_rx -> unconnected-(U13-Pad14)
- U13 pad 4: unconnected-(U13-Pad4) -> /gps_tx
- U13 pad 5: /gps_tx -> unconnected-(U13-Pad5)
- U4 pad 4: /s1_out_1 -> /s2_out_1
- U4 pad 5: /s2_out_1 -> /s1_out_1
- U4 pad 6: /s3_out_1 -> /s4_out_1
- U4 pad 7: /s4_out_1 -> /s3_out_1
- U5 pad 4: /s5_out_1 -> /s6_out_1
- U5 pad 5: /s6_out_1 -> /s5_out_1
- U5 pad 6: /s7_out_1 -> /s8_out_1
- U5 pad 7: /s8_out_1 -> /s7_out_1
- U6 pad 4: /s9_out_1 -> /s11_out_1
- U6 pad 5: /s10_out_1 -> /s14_out_1
- U6 pad 6: /s11_out_1 -> /s13_out_1
- U7 pad 4: /s13_out_1 -> /s10_out_1
- U7 pad 5: /s14_out_1 -> /s9_out_1
- U8 pad 1: /s2_en_1 -> /s8_en_1
- U8 pad 2: /s3_en_1 -> /s7_en_1
- U8 pad 3: /s4_en_1 -> /s6_en_1
- U8 pad 5: /s6_en_1 -> /s4_en_1
- U8 pad 6: /s7_en_1 -> /s3_en_1
- U8 pad 7: /s8_en_1 -> /s2_en_1
Routing:
- net /SDA1: track 0.00 -> 161.2 mm
- net /SCL1: track 0.00 -> 156.5 mm
- net /uart_mux_s0: track 0.00 -> 123.3 mm
- net /uart_mux_s1: track 0.00 -> 121.1 mm
- net Net-(Q4-Pad3): track 0.00 -> 55.9 mm
- net Net-(Q3-Pad3): track 0.00 -> 55.1 mm
- net Net-(Q5-Pad3): track 0.00 -> 52.9 mm
- net /sr_clk: track 0.00 -> 52.2 mm
- net /sr_clear: track 0.00 -> 50.6 mm
- net 4.2v: track 0.00 -> 42.5 mm
- net Net-(Q6-Pad3): track 0.00 -> 33.9 mm
- net /s5_en_1: track 0.00 -> 28.3 mm
- net Net-(Q9-Pad3): track 0.00 -> 28.0 mm
- net /s11_12_13_en_1: track 0.00 -> 26.4 mm
- net /s4_en_1: track 0.00 -> 24.6 mm
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
Commit message: board in progress1
Parts:
- removed U11: GY-GPS6MV2, super-met:GY-GPS6MV2
- moved REF** 16.8 mm to (271.3, 81.3)
- moved RN1 4.92 mm to (233.0, 68.8)
- moved U10 4.11 mm to (259.1, 135.4)
- moved U8 2.41 mm to (252.2, 88.1), turned to -90 degrees
- moved Q3 1.32 mm to (237.6, 72.1)
- moved U4 1.27 mm to (242.3, 74.4)
- moved RN3 1.27 mm to (210.7, 78.5)
- moved REF** 1.14 mm to (238.3, 75.2)
- moved Q4 0.85 mm to (237.6, 68.6)
Connections:
- U8 pad 5: /s4_en_1 -> /s2_en_1
- U8 pad 7: /s2_en_1 -> /s4_en_1
Routing:
- net /uart_mux_s0: track 123.3 -> 451.3 mm
- net 3.3v: track 0.00 -> 60.4 mm, vias 0 -> 10
- net 5.2v: track 0.00 -> 52.4 mm, vias 0 -> 11
- net Net-(U10-Pad14): track 0.00 -> 52.0 mm
- net /sr_latch: track 0.00 -> 50.2 mm
- net /s1_en_1: track 18.0 -> 63.7 mm
- net Net-(Q3-Pad3): track 55.1 -> 16.1 mm
- net Net-(Q4-Pad3): track 55.9 -> 20.6 mm
- net GND: track 6.47 -> 40.2 mm, vias 0 -> 9
- net /s5_en_1: track 28.3 -> 60.1 mm
- net /SDA1: track 161.2 -> 129.6 mm
- net Net-(Q6-Pad3): track 33.9 -> 3.38 mm
- net /SCL1: track 156.5 -> 132.8 mm
- net Net-(Q5-Pad3): track 52.9 -> 34.7 mm
- net /s8_en_1: track 7.53 -> 20.6 mm
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
Commit message: board in progress
Parts:
- added U11: GY-GPS6MV2, super-met:GY-GPS6MV2, F.Cu at (243.6, 30.7)
- moved JP1 113.3 mm to (322.3, 181.6)
- moved U9 44.5 mm to (129.5, 34.8)
- moved J8 38.3 mm to (193.8, 24.5)
- moved Q12 38.3 mm to (200.9, 31.5)
- moved Q11 38.3 mm to (200.9, 35.1)
- moved Q8 38.3 mm to (201.0, 42.6)
- moved RN3 38.3 mm to (206.9, 40.4)
- moved RN4 38.3 mm to (195.2, 47.6)
- moved RN5 38.3 mm to (208.0, 32.6)
- moved U13 38.3 mm to (193.0, 38.1)
- moved Q10 38.3 mm to (191.2, 45.2)
- moved Q7 38.3 mm to (200.9, 39.1)
- moved Q9 38.3 mm to (191.2, 48.8)
- moved REF** 38.3 mm to (197.9, 43.7)
- moved REF** 38.3 mm to (192.4, 30.3)
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Connections:
- RN2 pad 5: Net-(Q6-Pad3) -> Net-(Q5-Pad3)
- RN2 pad 6: /SDA2 -> /SCL2
- RN2 pad 7: Net-(Q5-Pad3) -> Net-(Q6-Pad3)
- RN2 pad 8: /SCL2 -> /SDA2
Routing:
- net /uart_mux_s0: track 451.3 -> 6.23 mm
- net /SCL1: track 132.8 -> 4.19 mm
- net /SDA1: track 129.6 -> 2.79 mm
- net /sim800_rst: track 0.00 -> 65.1 mm
- net /uart_mux_s1: track 112.3 -> 49.1 mm
- net /s1_en_1: track 63.7 -> 15.5 mm
- net 3.3v: track 60.4 -> 94.5 mm, vias 10 -> 18
- net Net-(Q5-Pad3): track 34.7 -> 2.19 mm
- net 5.2v: track 52.4 -> 79.7 mm, vias 11 -> 13
- net GND: track 40.2 -> 49.2 mm, vias 9 -> 10
- net /s3_out_1: track 2.72 -> 10.7 mm
- net /s4_out_1: track 3.40 -> 10.1 mm
- net Net-(JP1-Pad1): track 4.37 -> 0.00 mm
- net /SDA2: track 19.2 -> 16.7 mm
- net Net-(Q4-Pad3): track 20.6 -> 22.9 mm
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
Commit message: in progress
Parts:
- removed TP1, TP2, TP3, TP4: TestPoint, TestPoint:TestPoint_Pad_2.0x2.0mm
- moved U11 56.7 mm to (189.5, 47.8), turned to 90 degrees
- moved J8 40.2 mm to (209.3, 61.6)
- moved Q11 39.6 mm to (217.3, 71.1)
- moved RN3 39.6 mm to (223.3, 76.4)
- moved RN5 39.6 mm to (224.4, 68.7)
- moved Q12 39.6 mm to (217.3, 67.6)
- moved Q7 39.6 mm to (217.3, 75.2)
- moved REF** 39.6 mm to (214.3, 79.8)
- moved Q8 39.6 mm to (217.4, 78.7)
- moved RN4 39.6 mm to (211.7, 83.7)
- moved U13 39.6 mm to (209.5, 74.2)
- moved Q10 39.6 mm to (207.6, 81.3)
- moved Q9 39.6 mm to (207.6, 84.8)
- moved REF** 39.6 mm to (208.8, 66.3)
- moved U9 25.7 mm to (155.2, 35.8), turned to -90 degrees
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Routing:
- net /SCL1: track 4.19 -> 197.2 mm
- net /SDA1: track 2.79 -> 186.0 mm
- net /uart_mux_s0: track 6.23 -> 93.8 mm
- net /sr_in: track 0.00 -> 73.8 mm
- net /sim800_rst: track 65.1 -> 0.00 mm
- net /esp_rx: track 0.00 -> 61.2 mm
- net /esp_tx: track 0.00 -> 56.1 mm
- net /uart_mux_s1: track 49.1 -> 90.7 mm
- net Net-(Q3-Pad3): track 16.1 -> 54.6 mm
- net Net-(Q4-Pad3): track 22.9 -> 57.0 mm
- net Net-(Q6-Pad3): track 3.04 -> 34.4 mm
- net GND: track 49.2 -> 77.1 mm
- net Net-(Q5-Pad3): track 2.19 -> 28.8 mm
- net 3.3v: track 94.5 -> 117.4 mm, vias 18 -> 21
- net /s5_en_1: track 60.1 -> 41.0 mm
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
Commit message: board in progress
Parts:
- removed JP1: Jumper_2_Bridged, Jumper:SolderJumper-2_P1.3mm_Open_RoundedPad1.0x1.5mm
- removed the REF** at (295.4, 78.5)
- C1, C2, C3, C4, C6: moved to F.Cu
- moved C6 104.9 mm to (204.0, 74.0), turned to 90 degrees
- moved U9 90.9 mm to (228.1, 90.2), turned to 0 degrees
- moved C3 86.4 mm to (244.6, 74.4), turned to -90 degrees
- moved TP5 84.1 mm to (229.4, 126.2)
- moved R1 74.9 mm to (201.8, 125.5)
- moved R4 73.1 mm to (202.8, 122.2), turned to 90 degrees
- moved Q1 67.2 mm to (199.5, 122.2), turned to 180 degrees
- moved R3 66.3 mm to (200.3, 96.0), turned to -90 degrees
- moved Q2 59.0 mm to (199.9, 102.4), turned to 90 degrees
- moved R5 58.1 mm to (202.2, 104.1)
- moved C1 55.3 mm to (238.8, 105.5), turned to -90 degrees
- moved R2 52.6 mm to (198.9, 106.4), turned to 90 degrees
- moved U3 51.8 mm to (191.4, 102.4), turned to -90 degrees
- moved U1 49.8 mm to (192.0, 80.5), turned to -90 degrees
- moved U2 49.7 mm to (191.3, 128.5), turned to -90 degrees
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Routing:
- net GND: track 77.1 -> 540.9 mm, vias 10 -> 17
- net 5.2v: track 94.3 -> 355.1 mm, vias 14 -> 19
- net 3.3v: track 117.4 -> 351.2 mm, vias 21 -> 23
- net /Power_Vin: track 0.00 -> 83.3 mm, vias 0 -> 3
- net /uart_mux_rx: track 2.72 -> 85.1 mm, vias 0 -> 2
- net /uart_mux_tx: track 2.85 -> 69.4 mm, vias 0 -> 2
- net /sr_clear: track 48.0 -> 113.0 mm
- net /sr_latch: track 52.9 -> 107.3 mm
- net /sr_clk: track 50.6 -> 102.8 mm
- net /sim800_rst: track 0.00 -> 33.9 mm
- net 4.2v: track 42.5 -> 73.9 mm, vias 0 -> 1
- net /gps_tx: track 0.00 -> 31.3 mm
- net /en_5.2v_signal: track 0.00 -> 27.7 mm, vias 0 -> 1
- net Net-(Q8-Pad2): track 7.28 -> 28.8 mm
- net /s1_en_1: track 0.00 -> 19.6 mm, vias 0 -> 2
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Other:
- board size 99.1 x 99.1 mm -> 99.3 x 99.3 mm

Commit message: board in progress
Routing:
- net 3.3v: track 351.2 -> 307.8 mm
- net 5.2v: track 355.1 -> 356.3 mm, vias 19 -> 18

Commit message: board in progress
Parts:
- moved C2 7.03 mm to (245.3, 131.1), turned to 0 degrees
- moved C4 2.65 mm to (243.3, 123.1)
- moved C6 1.24 mm to (203.7, 72.8)
- moved C1 1.05 mm to (239.3, 106.4)
- moved C3 0.98 mm to (243.8, 75.0)
Routing:
- net /sr_latch: track 107.3 -> 14.4 mm
- net /sr_clk: track 102.8 -> 10.9 mm
- net /sr_clear: track 113.0 -> 51.3 mm
- net 3.3v: track 307.8 -> 357.1 mm
- net GND: track 541.0 -> 571.6 mm, vias 17 -> 18
- net 5.2v: track 356.3 -> 377.2 mm
- net Net-(Q4-Pad3): track 57.0 -> 66.1 mm
- net /uart_mux_s1: track 93.5 -> 98.7 mm
- net /sim800_rst: track 33.9 -> 37.9 mm
- net Net-(Q5-Pad3): track 28.8 -> 32.8 mm
- net 4.2v: track 73.9 -> 71.5 mm
- net Net-(Q9-Pad3): track 29.5 -> 31.8 mm
- net /SCL1: track 197.6 -> 199.5 mm
- net /s10_out_1: track 12.9 -> 14.4 mm
- net /s6_en_1: track 35.6 -> 34.3 mm
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
Commit message: before fill
Parts:
- moved U12 9.02 mm to (234.4, 145.8)
Routing:
- net /sr_clk: track 10.9 -> 130.6 mm
- net /sr_latch: track 14.4 -> 121.3 mm
- net /sr_clear: track 51.3 -> 123.6 mm
- net /SCL1: track 199.5 -> 223.1 mm
- net /SDA1: track 187.3 -> 209.1 mm
- net GND: track 571.6 -> 557.3 mm
- net Net-(Q4-Pad3): track 66.1 -> 75.2 mm
- net /esp_tx: track 56.1 -> 48.3 mm
- net 3.3v: track 357.1 -> 360.2 mm
- net Net-(U10-Pad14): track 52.7 -> 55.5 mm
- net 5.2v: track 377.2 -> 374.5 mm
- net /Power_Vin: track 83.3 -> 85.8 mm, vias 2 -> 3
- net /uart_mux_rx: track 84.7 -> 86.6 mm
- net Net-(Q3-Pad3): track 54.4 -> 56.1 mm
- net Net-(Q6-Pad3): track 35.3 -> 36.6 mm
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