File: super-met v6/super-met-v6/super-met-v6.kicad_pcb (KiCad board)
At the start: 2 copper layers, 99.3 x 99.3 mm, 57 parts, among them J1 Conn_01x02, J2 Conn_01x08, J3 Conn_01x08, J4 Conn_01x04, J5 Conn_01x08, J6 Conn_01x04, J7 Conn_01x02, J8 Conn_01x02, Q1 AO3400A, Q10 AO3400A, Q11 AO3400A, Q12 AO3400A, Q2 AO3400A, Q3 AO3400A, Q4 AO3400A, Q5 AO3400A, Q6 AO3400A, Q7 AO3400A, Q8 AO3400A, Q9 AO3400A, U1 DC-DC_MOD, U10 74HC595, U11 GY-GPS6MV2, U12 ESP-01v090, U13 74HC4052D, U14 BLUEPILL, U2 DC-DC_MOD, U3 DC-DC_MOD, U4 ADS1115IDGS, U5 ADS1115IDGS, U6 ADS1115IDGS, U7 ADS1115IDGS, U8 74HC595, U9 SIM800L

Commit message: filling
Routing:
- net /sr_clk: track 130.6 -> 50.6 mm
- net /sr_clear: track 123.6 -> 48.2 mm
- net 5.2v: track 374.5 -> 301.6 mm
- net /sr_latch: track 121.3 -> 52.7 mm
- net GND: track 557.3 -> 517.7 mm
- net /SDA1: track 209.1 -> 188.1 mm
- net /SCL1: track 223.1 -> 202.3 mm
- net 3.3v: track 360.2 -> 349.6 mm
- net Net-(U10-Pad14): track 55.5 -> 53.1 mm
- added copper zone on B.Cu, net (none)
- added copper zone on B.Cu, net /Power_Vin
- added copper zone on F.Cu, net /Power_Vin
- added copper zone on B.Cu, net 3.3v
- added copper zone on B.Cu, net 5.2v
- added copper zone on B.Cu, net GND
- added copper zone on F.Cu, net GND

Commit message: filled
Parts:
- moved H2 323.6 mm to (49.8, 110.5)
- moved H1 295.0 mm to (89.2, 52.1)
- moved H3 284.9 mm to (124.5, 26.2)
- moved C1 145.0 mm to (99.3, 68.3)
- moved C2 145.0 mm to (105.3, 93.0)
- moved C3 145.0 mm to (103.9, 36.9)
- moved C4 145.0 mm to (103.4, 85.0)
- moved C5 145.0 mm to (109.0, 57.1)
- moved C6 145.0 mm to (63.8, 34.7)
- moved J2 145.0 mm to (109.7, 43.4)
- moved J3 145.0 mm to (109.7, 75.2)
- moved J4 145.0 mm to (109.4, 80.0)
- moved J5 145.0 mm to (109.7, 106.6)
- moved J6 145.0 mm to (109.7, 111.0)
- moved J7 145.0 mm to (36.4, 95.3)
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Routing:
- net /sr_clk: track 50.6 -> 132.2 mm
- net /sr_clear: track 48.2 -> 124.4 mm
- net /sr_latch: track 52.7 -> 122.4 mm
- net GND: track 517.7 -> 527.9 mm
- net 3.3v: track 349.6 -> 352.9 mm, vias 23 -> 22
- net Net-(Q2-Pad1): track 5.60 -> 6.87 mm
- net 4.2v: track 71.5 -> 71.0 mm
- added copper zone on F.Cu, net 3.3v
- added copper zone on F.Cu, net 5.2v

Commit message: minor pcb fixes
Routing:
- net Net-(Q4-Pad3): track 75.2 -> 75.8 mm
- net 3.3v: track 352.9 -> 352.3 mm
- net /s1_out_1: track 11.9 -> 12.5 mm
- net /sr_latch: track 122.4 -> 122.9 mm

Commit message: preparing sensors board
Routing:
- net 5.2v: track 301.8 -> 303.4 mm
- net /gps_tx: track 31.5 -> 32.6 mm
- net /s8_en_1: track 22.3 -> 23.3 mm
- net /s7_en_1: track 28.9 -> 29.7 mm
- net /s6_en_1: track 34.5 -> 35.1 mm

Commit message: 4 layer init
Routing:
- net GND: track 527.9 -> 0.00 mm, vias 18 -> 0
- net 3.3v: track 352.6 -> 0.00 mm, vias 22 -> 0
- net 5.2v: track 303.4 -> 0.00 mm, vias 18 -> 0
- net /SCL1: track 202.3 -> 0.00 mm
- net /SDA1: track 188.1 -> 0.00 mm
- net /sr_clk: track 132.5 -> 0.00 mm, vias 2 -> 0
- net /sr_clear: track 124.4 -> 0.00 mm, vias 2 -> 0
- net /sr_latch: track 122.9 -> 0.00 mm, vias 2 -> 0
- net /uart_mux_s1: track 98.4 -> 0.00 mm
- net /uart_mux_s0: track 96.4 -> 0.00 mm
- net /uart_mux_rx: track 86.6 -> 0.00 mm, vias 2 -> 0
- net /Power_Vin: track 85.8 -> 0.00 mm, vias 3 -> 0
- net Net-(Q4-Pad3): track 75.8 -> 0.00 mm
- net /sr_in: track 74.1 -> 0.00 mm
- net 4.2v: track 71.0 -> 0.00 mm, vias 1 -> 0
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- removed copper zone on B.Cu, net (none)
- removed copper zone on B.Cu, net /Power_Vin
- removed copper zone on F.Cu, net /Power_Vin
- removed copper zone on B.Cu, net 3.3v
- removed copper zone on F.Cu, net 3.3v
- removed copper zone on B.Cu, net 5.2v
- removed copper zone on F.Cu, net 5.2v
- removed copper zone on B.Cu, net GND
- removed copper zone on F.Cu, net GND
Other:
- copper layers 2 -> 4

Commit message: in progress
Parts:
- removed REF** (x2): 0, Resistor_SMD:R_0603_1608Metric
- removed REF**: 0, Resistor_SMD:R_1206_3216Metric
- moved J1 8.37 mm to (34.9, 66.0), turned to 180 degrees
- moved RN5 3.70 mm to (81.0, 31.9)
- moved J7 3.40 mm to (33.0, 95.5), turned to 0 degrees
- moved RN3 2.39 mm to (81.0, 38.9)
- moved C3 1.69 mm to (105.4, 36.2)
- moved Q12 1.33 mm to (76.7, 30.6)
- moved Q11 1.33 mm to (76.7, 34.2)
- moved Q8 1.03 mm to (76.7, 41.3)
- moved Q7 0.93 mm to (76.7, 37.7)
- moved RN4 0.66 mm to (71.6, 45.0)
- moved C6 0.40 mm to (64.2, 34.7)
- moved Q9 0.27 mm to (67.6, 47.0)
- moved Q10 0.09 mm to (67.6, 43.2)
Connections:
- U12 pad 6: Net-(JP1-Pad1) -> unconnected-(U12-Pad6)
Routing:
- net 3.3v: track 0.00 -> 20.2 mm, vias 0 -> 1
- net /particles_tx: track 0.00 -> 18.5 mm
- net /particles_rx: track 0.00 -> 17.6 mm
- net Net-(Q9-Pad3): track 0.00 -> 15.5 mm
- net Net-(Q10-Pad3): track 0.00 -> 12.6 mm
- net Net-(Q11-Pad3): track 0.00 -> 10.1 mm
- net /sim800_tx: track 0.00 -> 9.59 mm
- net /sim800_rx: track 0.00 -> 9.05 mm
- net Net-(Q12-Pad3): track 0.00 -> 8.53 mm
- net GND: track 0.00 -> 5.85 mm
- net /uart_mux_tx: track 0.00 -> 3.78 mm
- net 5.2v: track 0.00 -> 3.77 mm, vias 0 -> 1
- net Net-(Q8-Pad2): track 0.00 -> 3.49 mm
- net /uart_mux_s0: track 0.00 -> 3.37 mm
- net Net-(Q7-Pad2): track 0.00 -> 2.62 mm
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
Commit message: before rearrange
Parts:
- Q3, Q4, Q5, Q6, RN1, RN2, U10, U8: moved to F.Cu
- moved C1 97.7 mm to (197.0, 66.7)
- moved TP5 90.3 mm to (179.7, 87.0)
- moved C2 82.8 mm to (184.9, 70.2)
- moved C4 82.8 mm to (183.0, 62.3)
- moved C5 52.4 mm to (161.3, 57.5)
- moved C6 36.9 mm to (42.5, 4.80)
- moved U8 20.2 mm to (101.9, 32.8), turned to 180 degrees
- moved C3 18.4 mm to (105.2, 17.8)
- moved U10 17.1 mm to (102.1, 96.0), turned to 180 degrees
- moved Q4 9.27 mm to (88.9, 33.7), turned to -90 degrees
- moved Q5 5.52 mm to (96.7, 81.7), turned to 180 degrees
- moved Q6 5.52 mm to (96.7, 78.1), turned to 180 degrees
- moved Q3 5.17 mm to (92.5, 33.7), turned to -90 degrees
- moved RN1 4.22 mm to (89.2, 29.1), turned to -90 degrees
- moved RN2 4.10 mm to (92.6, 80.0), turned to 0 degrees
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Connections:
- U10 pad 1: /s9_en_1 -> unconnected-(U10-Pad1)
- U10 pad 15: /s11_12_13_en_1 -> unconnected-(U10-Pad15)
- U10 pad 2: /s10_en_1 -> unconnected-(U10-Pad2)
- U10 pad 3: /s14_en_1 -> unconnected-(U10-Pad3)
- U10 pad 4: unconnected-(U10-Pad4) -> /s9_en_1
- U10 pad 5: unconnected-(U10-Pad5) -> /s10_en_1
- U10 pad 6: unconnected-(U10-Pad6) -> /s14_en_1
- U10 pad 7: unconnected-(U10-Pad7) -> /s11_12_13_en_1
- U14 pad 29: /sr_clear -> /sr_latch
- U14 pad 31: /sr_latch -> /sr_clear
- U6 pad 4: /s11_out_1 -> /s14_out_1
- U6 pad 5: /s14_out_1 -> /s11_out_1
- U8 pad 1: /s8_en_1 -> /s6_en_1
- U8 pad 15: /s1_en_1 -> /s5_en_1
- U8 pad 3: /s6_en_1 -> /s8_en_1
- U8 pad 4: /s5_en_1 -> /s1_en_1
Routing:
- net /uart_mux_s0: track 3.37 -> 80.9 mm, vias 0 -> 1
- net /uart_mux_s1: track 2.56 -> 79.7 mm, vias 0 -> 1
- net /SCL1: track 0.00 -> 63.5 mm
- net /esp_rx: track 0.00 -> 56.8 mm
- net /esp_tx: track 0.00 -> 48.8 mm
- net /SDA1: track 0.00 -> 47.2 mm
- net /s5_en_1: track 0.00 -> 46.4 mm
- net Net-(Q4-Pad3): track 0.00 -> 41.3 mm, vias 0 -> 1
- net Net-(Q3-Pad3): track 0.00 -> 39.2 mm, vias 0 -> 1
- net /s6_en_1: track 0.00 -> 35.7 mm
- net /s7_en_1: track 0.00 -> 34.4 mm
- net Net-(Q5-Pad3): track 0.00 -> 32.1 mm, vias 0 -> 1
- net Net-(Q6-Pad3): track 0.00 -> 32.0 mm, vias 0 -> 2
- net /gps_rx: track 0.00 -> 31.6 mm, vias 0 -> 1
- net /s8_en_1: track 0.00 -> 31.3 mm
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
Commit message: in progress
Parts:
- added JP1: Jumper_2_Bridged, Jumper:SolderJumper-2_P1.3mm_Open_TrianglePad1.0x1.5mm, F.Cu at (103.3, 106.6)
- C2, C3, C6: moved to B.Cu
- J7, J8: footprint Connector_JST:JST_XA_S02B-XASK-1N-BN_1x02_P2.50mm_Horizontal -> Connector_JST:JST_XA_B02B-XASK-1_1x02_P2.50mm_Vertical
- moved H3 102.2 mm to (24.6, 47.9)
- moved C1 91.9 mm to (105.2, 70.2), turned to 90 degrees
- moved C2 86.1 mm to (101.6, 91.9), turned to -90 degrees
- moved C4 79.8 mm to (105.8, 82.7)
- moved RN1 74.8 mm to (80.4, 103.4), turned to 90 degrees
- moved Q3 66.9 mm to (77.1, 98.8), turned to 90 degrees
- moved C5 65.9 mm to (97.9, 39.6)
- moved Q4 65.7 mm to (80.6, 98.8), turned to 90 degrees
- moved TP5 62.8 mm to (120.4, 107.7)
- moved C6 49.2 mm to (71.2, 44.7), turned to -90 degrees
- moved J7 32.0 mm to (61.4, 110.5)
- moved C3 28.1 mm to (105.4, 45.8), turned to 90 degrees
- moved U4 19.7 mm to (104.5, 51.9), turned to 90 degrees
- moved J1 18.3 mm to (48.7, 78.0)
- moved J8 17.1 mm to (83.8, 32.5), turned to 90 degrees
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Connections:
- C1 pad 2: GND -> GND3
- C2 pad 2: GND -> GND3
- C3 pad 2: GND -> GND3
- C4 pad 2: GND -> GND3
- J5 pad 1: GND -> GND3
- J6 pad 2: GND -> GND3
- U4 pad 1: GND -> GND3
- U4 pad 3: GND -> GND3
- U4 pad 4: /s2_out_1 -> /s1_out_1
- U4 pad 5: /s1_out_1 -> /s2_out_1
- U5 pad 3: GND -> GND3
- U6 pad 1: GND -> GND3
- U6 pad 3: GND -> GND3
- U6 pad 4: /s14_out_1 -> /s11_out_1
- U6 pad 5: /s11_out_1 -> unconnected-(U6-Pad5)
- U7 pad 3: GND -> GND3
Routing:
- net /sr_latch: track 0.00 -> 89.4 mm, vias 0 -> 1
- net /sr_clk: track 0.00 -> 88.8 mm, vias 0 -> 1
- net /uart_mux_rx: track 2.45 -> 86.2 mm, vias 0 -> 1
- net /sr_clear: track 0.00 -> 82.7 mm
- net Net-(U10-Pad14): track 0.00 -> 78.0 mm
- net /uart_mux_tx: track 3.78 -> 77.5 mm, vias 0 -> 1
- net /sr_in: track 0.00 -> 66.5 mm
- net GND: track 12.5 -> 65.9 mm, vias 0 -> 61
- net 5.2v: track 3.77 -> 51.3 mm, vias 1 -> 23
- net Net-(Q3-Pad3): track 39.2 -> 85.8 mm
- net Net-(Q4-Pad3): track 41.3 -> 82.1 mm, vias 1 -> 3
- net GND3: track 0.00 -> 35.5 mm, vias 0 -> 14
- net /en_4.2v_signal: track 0.00 -> 22.5 mm
- net 3.3v: track 20.2 -> 42.5 mm, vias 1 -> 26
- net /en_5.2v_signal: track 0.00 -> 21.3 mm
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- added copper zone on F.Cu, net /Power_Vin
- added copper zone on In1.Cu, net /Power_Vin
- added copper zone on F.Cu, net 3.3v
- added copper zone on F.Cu, net 4.2v
- added copper zone on In1.Cu, net 4.2v
- added copper zone on F.Cu, net 5.2v
- added copper zone on F.Cu, net GND
- added copper zone on In2.Cu, net GND
- added copper zone on F.Cu, net GND3
- added copper zone on In2.Cu, net GND3
Other:
- board size 99.3 x 99.3 mm -> 75.1 x 95.1 mm
