File: super-met v6/super-met-v6/super-met-v6.kicad_pcb (KiCad board)
At the start: 4 copper layers, 75.1 x 95.1 mm, 55 parts, among them J1 Conn_01x02, J2 Conn_01x08, J3 Conn_01x08, J4 Conn_01x04, J5 Conn_01x08, J6 Conn_01x04, J7 Conn_01x02, J8 Conn_01x02, Q1 AO3400A, Q10 AO3400A, Q11 AO3400A, Q12 AO3400A, Q2 AO3400A, Q3 AO3400A, Q4 AO3400A, Q5 AO3400A, Q6 AO3400A, Q7 AO3400A, Q8 AO3400A, Q9 AO3400A, U1 DC-DC_MOD, U10 74HC595, U11 GY-GPS6MV2, U12 ESP-01v090, U13 74HC4052D, U14 BLUEPILL, U2 DC-DC_MOD, U3 DC-DC_MOD, U4 ADS1115IDGS, U5 ADS1115IDGS, U6 ADS1115IDGS, U7 ADS1115IDGS, U8 74HC595, U9 SIM800L

Commit message: almost done?
Parts:
- removed H3: MountingHole, MountingHole:MountingHole_3.2mm_M3
- added ?: , , F.Cu at (56.9, 117.9)
- added ?: , , F.Cu at (68.6, 78.7)
- added ?: , , F.Cu at (91.4, 87.4)
- added ?: , , F.Cu at (91.4, 97.5)
- added TP1: TestPoint, TestPoint:TestPoint_Pad_2.0x2.0mm, F.Cu at (63.0, 117.9)
- added TP10: TestPoint, TestPoint:TestPoint_Pad_2.0x2.0mm, F.Cu at (68.6, 81.8)
- added TP11: TestPoint, TestPoint:TestPoint_Pad_2.0x2.0mm, F.Cu at (68.6, 84.8)
- added TP2: TestPoint, TestPoint:TestPoint_Pad_2.0x2.0mm, F.Cu at (59.9, 117.9)
- added TP3: TestPoint, TestPoint:TestPoint_Pad_2.0x2.0mm, F.Cu at (91.4, 100.1)
- added TP4: TestPoint, TestPoint:TestPoint_Pad_2.0x2.0mm, F.Cu at (91.4, 102.6)
- added TP6: TestPoint, TestPoint:TestPoint_Pad_2.0x2.0mm, F.Cu at (91.4, 105.7)
- added TP7: TestPoint, TestPoint:TestPoint_Pad_2.0x2.0mm, F.Cu at (91.4, 108.2)
- added TP8: TestPoint, TestPoint:TestPoint_Pad_2.0x2.0mm, F.Cu at (91.4, 78.7)
- added TP9: TestPoint, TestPoint:TestPoint_Pad_2.0x2.0mm, F.Cu at (91.4, 84.8)
- moved TP5 55.3 mm to (66.0, 117.9)
- moved C2 1.53 mm to (101.7, 93.5)
Routing:
- net 5.2v: track 51.3 -> 323.6 mm, vias 23 -> 25
- net 3.3v: track 42.5 -> 119.9 mm, vias 26 -> 31
- net 4.2v: track 0.00 -> 55.1 mm, vias 13 -> 14
- net /Power_Vin: track 0.00 -> 50.1 mm, vias 39 -> 44
- net /SCL1: track 60.4 -> 86.7 mm
- net /SDA1: track 60.3 -> 81.1 mm
- net GND: track 65.9 -> 76.2 mm, vias 61 -> 64
- net /uart_mux_s1: track 84.8 -> 89.0 mm
- net /uart_mux_s0: track 86.2 -> 90.4 mm
- net /uart_mux_tx: track 77.5 -> 81.5 mm
- net /uart_mux_rx: track 86.2 -> 90.2 mm
- net GND3: track 35.5 -> 39.4 mm
- net /esp_rx: track 71.4 -> 75.3 mm
- net /esp_tx: track 56.7 -> 60.4 mm
- net /SCL2: track 24.1 -> 25.2 mm
- added copper zone on B.Cu, net (none)
- added copper zone on F.Cu, net (none)
- added copper zone on In1.Cu, net 3.3v
- added copper zone on In1.Cu, net 5.2v
- added copper zone on B.Cu, net GND
- removed copper zone on In1.Cu, net 4.2v

Commit message: almost done ?
Routing:
- net GND: track 76.2 -> 155.2 mm
- net /Power_Vin: track 50.1 -> 73.5 mm
- net 3.3v: track 119.9 -> 128.2 mm
- net 5.2v: track 323.6 -> 331.6 mm
- net 4.2v: track 55.1 -> 62.9 mm
- removed copper zone on F.Cu, net /Power_Vin
- removed copper zone on F.Cu, net 3.3v
- removed copper zone on F.Cu, net 4.2v
- removed copper zone on F.Cu, net 5.2v

Commit message: before_changing_fills
Parts:
- removed ? (x4): , 
Connections:
- R3 pad 2: 4.2v -> GND
Routing:
- net 4.2v: track 62.9 -> 60.3 mm, vias 14 -> 13

Commit message: before_changing_fills
Parts:
- added ?: , , F.Cu at (56.9, 117.9)
- added ?: , , F.Cu at (68.6, 78.7)
- added ?: , , F.Cu at (91.4, 87.4)
- added ?: , , F.Cu at (91.4, 97.5)
Routing:
- net GND: track 155.2 -> 128.4 mm, vias 64 -> 49
- net unconnected-(U6-Pad5): track 12.4 -> 0.00 mm
- net /s14_out_1: track 0.00 -> 12.4 mm

Commit message: ready for order
Parts:
- D->A Grounds: renamed from JP1
- H1 M3: renamed from H1
- H2 M3: renamed from H2
- renumbered TP5 to 3.3v, TP10 to Esp_rx, TP11 to Esp_tx, TP2 to SCL, TP9 to SCL2, TP1 to SDA, TP8 to SDA2, TP3 to u_rx, TP7 to u_s0, TP6 to u_s1, TP4 to u_tx
Routing:
- net /Power_Vin: track 73.5 -> 38.8 mm, vias 44 -> 39
- net GND: track 128.4 -> 103.6 mm, vias 49 -> 59
- net 3.3v: track 128.2 -> 117.9 mm, vias 31 -> 29
- net 5.2v: track 331.6 -> 323.4 mm, vias 25 -> 130
- net 4.2v: track 60.3 -> 53.4 mm
- net /sr_in: track 66.5 -> 68.0 mm
- net /en_5.2v: track 3.01 -> 3.65 mm
- net /gps_tx: track 11.0 -> 11.5 mm
- added copper zone on B.Cu, net /Power_Vin
- added copper zone on F.Cu, net /Power_Vin
- added copper zone on F.Cu, net 3.3v
- added copper zone on F.Cu, net 4.2v
- added copper zone on F.Cu, net 5.2v
- removed copper zone on B.Cu, net (none)
- removed copper zone on F.Cu, net (none)
Other:
- board text added: "5.2v"
- board text added: "<-sr_clk"
- board text added: "<-sr_clr"
- board text added: "<-sr_data"
- board text added: "<-sr_latch"
- board text added: "Gnd"
- board text added: "Super-met v0.1"
- board text added: "V&V Design"
- board text added: "en_4.2v"
- board text added: "en_5.2v"
- board text added: "gnd"
- board text added: "particles_rx"
- board text added: "particles_tx"
- board text added: "sim800_rst"
- board text added: "vin"

Commit message: ready for order
Parts:
- renumbered SDA2 to <-SDA2
Routing:
- net GND: track 103.6 -> 104.8 mm
Other:
- board text added: "3.3v"
- board text added: "4.2v"
- board text added: "Esp_rx"
- board text added: "Esp_tx"
- board text added: "RST CH_PD 3.3v"
- board text added: "Vin"
- board text added: "scl1"
- board text added: "sda1"
