File: super-met v6/super-met-v6/super-met-v6.kicad_sch (KiCad schematic)
At the start: 6 parts

Commit message: main scheme:
Parts:
- added C?: C_Small, symbol Device:C_Small
- added C? (x6): 0.1uF, symbol Device:C_Small
- added H? (x3): MountingHole, symbol Mechanical:MountingHole
- added J? (x2): Conn_01x02, symbol Connector_Generic:Conn_01x02
- added JP?: Jumper_2_Bridged, symbol Jumper:Jumper_2_Bridged
- added Q? (x12): AO3400A, Package_TO_SOT_SMD:SOT-23, symbol Transistor_FET:AO3400A
- added R? (x2): 1k, symbol Device:R_Small
- added R? (x2): 100, symbol Device:R_Small
- added R?: R_Small, symbol Device:R_Small
- added RN? (x5): R_Pack04, symbol Device:R_Pack04
- added TP? (x5): TestPoint, symbol Connector:TestPoint
- added U? (x4): ADS1115IDGS, Package_SO:TSSOP-10_3x3mm_P0.5mm, symbol Analog_ADC:ADS1115IDGS
- added U?: GY-GPS6MV2, symbol super-met:GY-GPS6MV2
- added U?: SIM800L, symbol super-met:SIM800L
- added U? (x2): 74HC595, symbol 74xx:74HC595
- added U?: ESP-01v090, symbol ESP8266:ESP-01v090
- added U?: BLUEPILL, symbol super-met:BLUEPILL
- added U?: 74HC4052D, SOIC127P600X175-16N, symbol 74HC4052D:74HC4052D
Connections:
- net 3.3v: now also C?.1, Q?.1 (G), Q?.1 (G), Q?.1 (G), Q?.1 (G), Q?.1 (G), Q?.1 (G), Q?.1 (G), Q?.1 (G), Q?.1 (G), Q?.1 (G), RN?.3 (R3.1), RN?.3 (R3.1), RN?.4 (R4.1), RN?.4 (R4.1), RN?.5 (R4.2), RN?.6 (R3.2), RN?.7 (R2.2), RN?.7 (R2.2), RN?.8 (R1.2), RN?.8 (R1.2), TP?.1, U?.16 (VCC), U?.16 (VCC), U?.20 (3V3), U?.3 (CH_PD), U?.38 (3V3), U?.5 (RST), U?.7 (VCC)
- net 4.2v: now also U?.2 (Vcc)
- net 5.2v: now also C?.1, C?.1, C?.1, C?.1, C?.1, J?.1 (Pin_1), RN?.1 (R1.1), RN?.1 (R1.1), RN?.2 (R2.1), RN?.2 (R2.1), RN?.5 (R4.2), RN?.5 (R4.2), RN?.6 (R3.2), RN?.6 (R3.2), RN?.7 (R2.2), RN?.8 (R1.2), U?.1 (ADDR), U?.1 (ADDR), U?.1 (Vin), U?.16 (VCC), U?.8 (VDD), U?.8 (VDD), U?.8 (VDD), U?.8 (VDD)
- net en_4.2v: now also Q?.3 (D)
- net en_5.2v: now also Q?.3 (D)
- net Power_gnd renamed GND
- net GND: now also C?.2, C?.2, C?.2, C?.2, C?.2, C?.2, J?.2 (Pin_2), JP?.2 (B), Q?.2 (S), Q?.2 (S), R?.2, R?.2, U?.1 (ADDR), U?.1 (ADDR), U?.13 (~{OE}), U?.13 (~{OE}), U?.19 (GND), U?.2 (GND), U?.3 (GND), U?.3 (GND), U?.3 (GND), U?.3 (GND), U?.39 (GND), U?.4 (Gnd), U?.40 (GND), U?.6 (Gnd), U?.6 (~E), U?.8 (GND), U?.8 (GND), U?.8 (GND)
- new net: JP?.1 (A), U?.6 (GPIO0)
- new net: Q?.3 (D), RN?.8 (R1.2), U?.10 (SCL), U?.10 (SCL) (x2)
- new net: Q?.3 (D), RN?.7 (R2.2), U?.9 (SDA), U?.9 (SDA) (x2)
- new net: Q?.3 (D), RN?.4 (R4.1), U?.9 (S1)
- new net: Q?.2 (S), RN?.3 (R3.1), U?.4 (Rx)
- new net: Q?.2 (S), RN?.4 (R4.1), U?.5 (Tx)
- new net: Q?.1 (G), R?.1, R?.2 (x2)
- new net: Q?.3 (D), RN?.4 (R4.1), U?.3 (2Z)
- new net: Q?.3 (D), RN?.3 (R3.1), U?.10 (S0)
- new net: Q?.3 (D), RN?.3 (R3.1), U?.13 (1Z)
- new net: U?.14 (SER), U?.9 (QH')
- new net SCL1: Q?.2 (S), RN?.6 (R3.2), U?.14 (PB6)
- new net SCL2: Q?.2 (S), RN?.6 (R3.2), U?.35 (PB10)
- new net SDA1: Q?.2 (S), RN?.5 (R4.2), U?.15 (PB7)
- new net SDA2: Q?.2 (S), RN?.5 (R4.2), U?.36 (PB11)
- new net en_4.2v_signal: R?.1, U?.3 (PB14)
- new net en_5.2v_signal: R?.1, U?.2 (PB13)
- new net esp_rx: TP?.1, U?.6 (PA9), U?.8 (URXD)
- new net esp_tx: TP?.1, U?.1 (UTXD), U?.7 (PA10)
- new net gps_rx: U?.14 (1Y1), U?.2 (Rx)
- new net gps_tx: U?.3 (Tx), U?.5 (2Y1)
- new net particles_rx: J?.1 (Pin_1), U?.15 (1Y2)
- new net particles_tx: J?.2 (Pin_2), U?.2 (2Y2)
- new net sim800_rst: U?.3 (Rst), U?.4 (PB15)
- new net sim800_rx: Q?.3 (D), RN?.2 (R2.1), U?.12 (1Y0)
- new net sim800_tx: Q?.3 (D), RN?.1 (R1.1), U?.1 (2Y0)
- new net sr_clear: U?.10 (~{SRCLR}), U?.10 (~{SRCLR}), U?.29 (PA4)
- new net sr_clk: U?.11 (SRCLK), U?.11 (SRCLK), U?.30 (PA5)
- new net sr_in: U?.14 (SER), U?.32 (PA7)
- new net sr_latch: U?.12 (RCLK), U?.12 (RCLK), U?.31 (PA6)
- new net uart_mux_rx: Q?.2 (S), RN?.1 (R1.1), TP?.1, U?.28 (PA3)
- new net uart_mux_s0: Q?.2 (S), RN?.2 (R2.1), U?.25 (PA0)
- new net uart_mux_s1: Q?.2 (S), RN?.1 (R1.1), U?.26 (PA1)
- new net uart_mux_tx: Q?.2 (S), RN?.2 (R2.1), TP?.1, U?.27 (PA2)
- no-connect marks 6 -> 36
Other:
- added sheet Sensors (sensors.kicad_sch)
- note added: "0x48"
- note added: "0x49"
- note added: "3.3v"
- note added: "4.2v"
- note added: "5.2v"
- note added: "rx"
- note added: "tx"

Commit message: sensors board
Parts:
- removed C?: C_Small, symbol Device:C_Small
- removed R? (x2): R_Small, symbol Device:R_Small
- added J2, J3, J5: Conn_01x08, Connector_JST:JST_PH_S8B-PH-K_1x08_P2.00mm_Horizontal, symbol Connector_Generic:Conn_01x08
- added J4, J6: Conn_01x04, Connector_PinHeader_2.54mm:PinHeader_1x04_P2.54mm_Horizontal, symbol Connector_Generic:Conn_01x04
- C1, C2, C3, C4, C5, C6: renamed from C?; footprint (none) -> Capacitor_SMD:C_0603_1608Metric_Pad1.08x0.95mm_HandSolder
- H1, H2, H3: renamed from H?; footprint (none) -> MountingHole:MountingHole_3.2mm_M3
- J1: renamed from J?; footprint (none) -> Connector_JST:JST_XA_B02B-XASK-1_1x02_P2.50mm_Vertical
- J7, J8: renamed from J?; footprint (none) -> Connector_JST:JST_XA_S02B-XASK-1N-BN_1x02_P2.50mm_Horizontal
- JP1: renamed from JP?; footprint (none) -> Jumper:SolderJumper-2_P1.3mm_Open_RoundedPad1.0x1.5mm
- R1, R2, R3, R4, R5: renamed from R?; footprint (none) -> Resistor_SMD:R_0805_2012Metric_Pad1.20x1.40mm_HandSolder
- RN1, RN2, RN3, RN4, RN5: renamed from RN?; footprint (none) -> Resistor_SMD:R_Array_Concave_4x0603
- TP1, TP2, TP3, TP4, TP5: renamed from TP?; footprint (none) -> TestPoint:TestPoint_Pad_2.0x2.0mm
- U1, U2, U3: renamed from U?; footprint (none) -> super-met:DC-DC
- U10, U8: renamed from U?; footprint (none) -> libs:SOIC127P600X175-16N
- U11: renamed from U?; footprint (none) -> super-met:GY-GPS6MV2
- U12: renamed from U?; footprint (none) -> ESP8266:ESP-01
- U13: renamed from U?; footprint SOIC127P600X175-16N -> libs:SOIC127P600X175-16N
- U14: renamed from U?; footprint (none) -> super-met:BLUEPILL
- U9: renamed from U?; footprint (none) -> super-met:SIM800L
- gave numbers to parts that had none: 16
Connections:
- net 3.3v: now also J6.1 (Pin_1)
- net 5.2v: now also J5.2 (Pin_2)
- net GND: now also J5.1 (Pin_1), J6.2 (Pin_2)
- net SCL1: now also J6.4 (Pin_4)
- net SDA1: now also J6.3 (Pin_3)
- net s1_out_1: now reaches U4.4 (AIN0)
- net s1_out_1: now also J2.1 (Pin_1)
- net s2_out_1: now reaches U4.5 (AIN1)
- net s2_out_1: now also J2.3 (Pin_3)
- net s3_out_1: now reaches U4.6 (AIN2)
- net s3_out_1: now also J2.5 (Pin_5)
- net s4_out_1: now reaches U4.7 (AIN3)
- net s4_out_1: now also J2.7 (Pin_7)
- net s5_out_1: now reaches U5.4 (AIN0)
- net s5_out_1: now also J3.1 (Pin_1)
- net s6_out_1: now reaches U5.5 (AIN1)
- net s6_out_1: now also J3.3 (Pin_3)
- net s7_out_1: now reaches U5.6 (AIN2)
- net s7_out_1: now also J3.5 (Pin_5)
- net s8_out_1: now reaches U5.7 (AIN3)
- net s8_out_1: now also J3.7 (Pin_7)
- net s9_out_1: now reaches U6.4 (AIN0)
- net s9_out_1: now also J5.3 (Pin_3)
- net s10_out_1: now reaches U6.5 (AIN1)
- net s10_out_1: now also J5.6 (Pin_6)
- net s11_out_1: now reaches U6.6 (AIN2)
- net s11_out_1: now also J4.4 (Pin_4)
- net s12_out_1: now reaches U6.7 (AIN3)
- net s12_out_1: now also J4.3 (Pin_3)
- net s13_out_1: now reaches U7.4 (AIN0)
- net s13_out_1: now also J4.2 (Pin_2)
- net s14_out_1: now reaches U7.5 (AIN1)
- net s14_out_1: now also J5.7 (Pin_7)
- net s10_en_1: now reaches U10.1 (QB)
- net s10_en_1: now also J5.5 (Pin_5)
- net s9_en_1: now reaches U10.15 (QA)
- net s9_en_1: now also J5.4 (Pin_4)
- net s14_en_1: now reaches U10.2 (QC)
- net s14_en_1: now also J5.8 (Pin_8)
- net s11_12_13_en_1: now reaches U10.3 (QD)
- net s11_12_13_en_1: now also J4.1 (Pin_1)
- net s2_en_1: now reaches U8.1 (QB)
- net s2_en_1: now also J2.4 (Pin_4)
- net s1_en_1: now reaches U8.15 (QA)
- net s1_en_1: now also J2.2 (Pin_2)
- net s3_en_1: now reaches U8.2 (QC)
- net s3_en_1: now also J2.6 (Pin_6)
- net s4_en_1: now reaches U8.3 (QD)
- net s4_en_1: now also J2.8 (Pin_8)
- net s5_en_1: now reaches U8.4 (QE)
- net s5_en_1: now also J3.2 (Pin_2)
- net s6_en_1: now reaches U8.5 (QF)
- net s6_en_1: now also J3.4 (Pin_4)
- net s7_en_1: now reaches U8.6 (QG)
- net s7_en_1: now also J3.6 (Pin_6)
- net s8_en_1: now reaches U8.7 (QH)
- net s8_en_1: now also J3.8 (Pin_8)
- no-connect marks 36 -> 49
Other:
- removed sheet Sensors

Commit message: board in progress
Connections:
- net 3.3v: now also RN1.2 (R2.1), RN2.1 (R1.1), RN3.8 (R1.2), RN4.6 (R3.2), RN5.6 (R3.2); no longer RN1.3 (R3.1), RN2.4 (R4.1), RN3.5 (R4.2), RN4.7 (R2.2), RN5.7 (R2.2)
- net 5.2v: now also RN1.3 (R3.1), RN2.4 (R4.1), RN3.5 (R4.2), RN4.7 (R2.2), RN5.7 (R2.2); no longer RN1.2 (R2.1), RN2.1 (R1.1), RN3.8 (R1.2), RN4.6 (R3.2), RN5.6 (R3.2)
- net SCL1: now also RN1.7 (R2.2); no longer RN1.6 (R3.2)
- net SCL2: now also RN2.8 (R1.2); no longer RN2.6 (R3.2)
- net SDA2: now also RN2.6 (R3.2); no longer RN2.5 (R4.2)
- net gps_rx: now also U13.11 (1Y3); no longer U13.14 (1Y1)
- net gps_tx: now also U13.4 (2Y3); no longer U13.5 (2Y1)
- net s10_en_1: now also U10.2 (QC); no longer U10.1 (QB)
- net s10_out_1: now also U7.4 (AIN0); no longer U6.5 (AIN1)
- net s11_12_13_en_1: now also U10.15 (QA); no longer U10.3 (QD)
- net s11_out_1: now also U6.4 (AIN0); no longer U6.6 (AIN2)
- net s13_out_1: now also U6.6 (AIN2); no longer U7.4 (AIN0)
- net s14_en_1: now also U10.3 (QD); no longer U10.2 (QC)
- net s14_out_1: now also U6.5 (AIN1); no longer U7.5 (AIN1)
- net s1_out_1: now also U4.5 (AIN1); no longer U4.4 (AIN0)
- net s2_en_1: now also U8.7 (QH); no longer U8.1 (QB)
- net s2_out_1: now also U4.4 (AIN0); no longer U4.5 (AIN1)
- net s3_en_1: now also U8.6 (QG); no longer U8.2 (QC)
- net s3_out_1: now also U4.7 (AIN3); no longer U4.6 (AIN2)
- net s4_en_1: now also U8.5 (QF); no longer U8.3 (QD)
- net s4_out_1: now also U4.6 (AIN2); no longer U4.7 (AIN3)
- net s5_out_1: now also U5.5 (AIN1); no longer U5.4 (AIN0)
- net s6_en_1: now also U8.3 (QD); no longer U8.5 (QF)
- net s6_out_1: now also U5.4 (AIN0); no longer U5.5 (AIN1)
- net s7_en_1: now also U8.2 (QC); no longer U8.6 (QG)
- net s7_out_1: now also U5.7 (AIN3); no longer U5.6 (AIN2)
- net s8_en_1: now also U8.1 (QB); no longer U8.7 (QH)
- net s8_out_1: now also U5.6 (AIN2); no longer U5.7 (AIN3)
- net s9_en_1: now also U10.1 (QB); no longer U10.15 (QA)
- net s9_out_1: now also U7.5 (AIN1); no longer U6.4 (AIN0)
- net sim800_rx: now also RN3.4 (R4.1); no longer RN3.2 (R2.1)
- net sim800_tx: now also RN3.2 (R2.1); no longer RN3.1 (R1.1)
- net uart_mux_rx: now also RN4.3 (R3.1); no longer RN4.1 (R1.1)
- net uart_mux_s0: now also RN5.1 (R1.1); no longer RN5.2 (R2.1)
- net uart_mux_s1: now also RN5.3 (R3.1); no longer RN5.1 (R1.1)
- net uart_mux_tx: now also RN4.1 (R1.1); no longer RN4.2 (R2.1)
- net at Q4.3 (D), U4.9 (SDA), U5.9 (SDA): now also RN1.6 (R3.2); no longer RN1.7 (R2.2)
- net at Q5.3 (D), U6.10 (SCL), U7.10 (SCL): now also RN2.7 (R2.2); no longer RN2.8 (R1.2)
- net at Q6.3 (D), U6.9 (SDA), U7.9 (SDA): now also RN2.5 (R4.2); no longer RN2.7 (R2.2)
- net at Q8.2 (S), U9.5 (Tx): now also RN3.1 (R1.1); no longer RN3.4 (R4.1)
- net at Q11.3 (D), U13.10 (S0): now also RN5.2 (R2.1); no longer RN5.3 (R3.1)
- net at Q9.3 (D), U13.13 (1Z): now also RN4.2 (R2.1); no longer RN4.3 (R3.1)
Other:
- note added: "поправлено под рез n"

Commit message: board in progress1
Connections:
- net s2_en_1: now also U8.5 (QF); no longer U8.7 (QH)
- net s4_en_1: now also U8.7 (QH); no longer U8.5 (QF)
Changed lines of the file:
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@@
     (effects (font (size 1.27 1.27)) (justify right bottom))
+  )
+  (label "s4_en_1" (at 224.79 153.67 0)
+    (effects (font (size 1.27 1.27)) (justify left bottom))
   )
   (label "SDA1" (at 163.83 45.72 0)
@@
     (effects (font (size 1.27 1.27)) (justify right bottom))
   )
+  (label "s2_en_1" (at 224.79 148.59 0)
+    (effects (font (size 1.27 1.27)) (justify left bottom))
+  )
   (label "uart_mux_tx" (at 48.26 179.07 0)
     (effects (font (size 1.27 1.27)) (justify left bottom))
@@
     (effects (font (size 1.27 1.27)) (justify left bottom))
   )
-  (label "s2_en_1" (at 224.79 153.67 0)
-    (effects (font (size 1.27 1.27)) (justify left bottom))
-  )
   (label "s10_en_1" (at 86.36 256.54 0)
     (effects (font (size 1.27 1.27)) (justify left bottom))
@@
     (effects (font (size 1.27 1.27)) (justify right bottom))
   )
-  (label "s4_en_1" (at 224.79 148.59 0)
-    (effects (font (size 1.27 1.27)) (justify left bottom))
-  )
   (label "s4_out_1" (at 86.36 180.34 0)

Commit message: board in progress
Connections:
- net SCL2: now also RN2.6 (R3.2); no longer RN2.8 (R1.2)
- net SDA2: now also RN2.8 (R1.2); no longer RN2.6 (R3.2)
- net at Q5.3 (D), U6.10 (SCL), U7.10 (SCL): now also RN2.5 (R4.2); no longer RN2.7 (R2.2)
- net at Q6.3 (D), U6.9 (SDA), U7.9 (SDA): now also RN2.7 (R2.2); no longer RN2.5 (R4.2)
Changed lines of the file:
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@@
+    (stroke (width 0) (type default) (color 0 0 0 0))
+  )
+  (wire (pts (xy 149.86 123.19) (xy 152.4 123.19))
     (stroke (width 0) (type default) (color 0 0 0 0))
   )
@@
     (stroke (width 0) (type default) (color 0 0 0 0))
   )
-  (wire (pts (xy 163.83 121.92) (xy 163.83 116.84))
+  (wire (pts (xy 163.83 116.84) (xy 163.83 128.27))
     (stroke (width 0) (type default) (color 0 0 0 0))
   )
@@
     (stroke (width 0) (type default) (color 0 0 0 0))
   )
-  (wire (pts (xy 157.48 120.65) (xy 157.48 121.92))
+  (wire (pts (xy 157.48 120.65) (xy 157.48 123.19))
     (stroke (width 0) (type default) (color 0 0 0 0))
   )
@@
     (stroke (width 0) (type default) (color 0 0 0 0))
   )
-  (wire (pts (xy 147.32 123.19) (xy 154.94 123.19))
-    (stroke (width 0) (type default) (color 0 0 0 0))
-  )
   (wire (pts (xy 227.33 73.66) (xy 227.33 76.2))
     (stroke (width 0) (type default) (color 0 0 0 0))
@@
     (stroke (width 0) (type default) (color 0 0 0 0))
   )
+  (wire (pts (xy 154.94 119.38) (xy 148.59 119.38))
+    (stroke (width 0) (type default) (color 0 0 0 0))
+  )
   (wire (pts (xy 158.75 52.07) (xy 162.56 52.07))
     (stroke (width 0) (type default) (color 0 0 0 0))
@@
     (stroke (width 0) (type default) (color 0 0 0 0))
   )
-  (wire (pts (xy 147.32 105.41) (xy 147.32 123.19))
+  (wire (pts (xy 147.32 105.41) (xy 147.32 121.92))
     (stroke (width 0) (type default) (color 0 0 0 0))
   )
@@
     (stroke (width 0) (type default) (color 0 0 0 0))
   )
-  (wire (pts (xy 158.75 123.19) (xy 158.75 121.92))
-    (stroke (width 0) (type default) (color 0 0 0 0))
-  )
   (wire (pts (xy 261.62 91.44) (xy 242.57 91.44))
     (stroke (width 0) (type default) (color 0 0 0 0))
@@
     (stroke (width 0) (type default) (color 0 0 0 0))
   )
+  (wire (pts (xy 149.86 128.27) (xy 149.86 123.19))
+    (stroke (width 0) (type default) (color 0 0 0 0))
+  )
   (wire (pts (xy 57.15 31.75) (xy 62.23 31.75))
     (stroke (width 0) (type default) (color 0 0 0 0))
@@
     (stroke (width 0) (type default) (color 0 0 0 0))
   )
+  (wire (pts (xy 160.02 123.19) (xy 160.02 121.92))
+    (stroke (width 0) (type default) (color 0 0 0 0))
+  )
   (wire (pts (xy 238.76 88.9) (xy 238.76 99.06))
     (stroke (width 0) (type default) (color 0 0 0 0))
@@
     (stroke (width 0) (type default) (color 0 0 0 0))
   )
+  (wire (pts (xy 163.83 128.27) (xy 149.86 128.27))
+    (stroke (width 0) (type default) (color 0 0 0 0))
+  )
   (polyline (pts (xy 16.51 20.32) (xy 68.58 20.32))
     (stroke (width 0) (type default) (color 0 0 0 0))
@@
     (stroke (width 0) (type default) (color 0 0 0 0))
   )
+  (wire (pts (xy 154.94 119.38) (xy 154.94 123.19))
+    (stroke (width 0) (type default) (color 0 0 0 0))
+  )
   (wire (pts (xy 160.02 134.62) (xy 154.94 134.62))
     (stroke (width 0) (type default) (color 0 0 0 0))
@@
     (stroke (width 0) (type default) (color 0 0 0 0))
   )
-  (wire (pts (xy 152.4 121.92) (xy 152.4 123.19))
-    (stroke (width 0) (type default) (color 0 0 0 0))
-  )
   (wire (pts (xy 144.78 36.83) (xy 144.78 45.72))
     (stroke (width 0) (type default) (color 0 0 0 0))
@@
     (stroke (width 0) (type default) (color 0 0 0 0))
   )
-  (wire (pts (xy 157.48 123.19) (xy 158.75 123.19))
-    (stroke (width 0) (type default) (color 0 0 0 0))
-  )
   (wire (pts (xy 201.93 44.45) (xy 201.93 50.8))
     (stroke (width 0) (type default) (color 0 0 0 0))
@@
     (stroke (width 0) (type default) (color 0 0 0 0))
   )
-  (wire (pts (xy 160.02 123.19) (xy 160.02 119.38))
-    (stroke (width 0) (type default) (color 0 0 0 0))
-  )
   (wire (pts (xy 27.94 111.76) (xy 30.48 111.76))
     (stroke (width 0) (type default) (color 0 0 0 0))
@@
     (stroke (width 0) (type default) (color 0 0 0 0))
   )
-  (wire (pts (xy 157.48 121.92) (xy 152.4 121.92))
-    (stroke (width 0) (type default) (color 0 0 0 0))
-  )
   (wire (pts (xy 128.27 90.17) (xy 128.27 92.71))
     (stroke (width 0) (type default) (color 0 0 0 0))
@@
     (stroke (width 0) (type default) (color 0 0 0 0))
   )
-  (wire (pts (xy 158.75 121.92) (xy 163.83 121.92))
-    (stroke (width 0) (type default) (color 0 0 0 0))
-  )
   (wire (pts (xy 228.6 91.44) (xy 228.6 101.6))
     (stroke (width 0) (type default) (color 0 0 0 0))
@@
     (stroke (width 0) (type default) (color 0 0 0 0))
   )
+  (wire (pts (xy 147.32 121.92) (xy 160.02 121.92))
+    (stroke (width 0) (type default) (color 0 0 0 0))
+  )
   (wire (pts (xy 153.67 62.23) (xy 153.67 63.5))
     (stroke (width 0) (type default) (color 0 0 0 0))
@@
     (stroke (width 0) (type default) (color 0 0 0 0))
   )
-  (wire (pts (xy 160.02 119.38) (xy 148.59 119.38))
-    (stroke (width 0) (type default) (color 0 0 0 0))
-  )
