File: super-met v6/super-met-v6/super-met-v6.kicad_sch (KiCad schematic)
At the start: 59 parts, among them J1 Conn_01x02, J2 Conn_01x08, J3 Conn_01x08, J4 Conn_01x04, J5 Conn_01x08, J6 Conn_01x04, J7 Conn_01x02, J8 Conn_01x02, Q1 AO3400A, Q10 AO3400A, Q11 AO3400A, Q12 AO3400A, Q2 AO3400A, Q3 AO3400A, Q4 AO3400A, Q5 AO3400A, Q6 AO3400A, Q7 AO3400A, Q8 AO3400A, Q9 AO3400A, U1 DC-DC_MOD, U10 74HC595, U11 GY-GPS6MV2, U12 ESP-01v090, U13 74HC4052D, U14 BLUEPILL, U2 DC-DC_MOD, U3 DC-DC_MOD, U4 ADS1115IDGS, U5 ADS1115IDGS, U6 ADS1115IDGS, U7 ADS1115IDGS, U8 74HC595, U9 SIM800L

Commit message: board in progress
Parts:
- removed JP1: Jumper_2_Bridged, Jumper:SolderJumper-2_P1.3mm_Open_RoundedPad1.0x1.5mm, symbol Jumper:Jumper_2_Bridged
- removed TP1, TP2, TP3, TP4: TestPoint, TestPoint:TestPoint_Pad_2.0x2.0mm, symbol Connector:TestPoint
Connections:
- no-connect marks 49 -> 50
Changed lines of the file:
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@@
   (junction (at 198.12 63.5) (diameter 0) (color 0 0 0 0)
   )
-  (junction (at 283.21 34.29) (diameter 0) (color 0 0 0 0)
-  )
   (junction (at 139.7 34.29) (diameter 0) (color 0 0 0 0)
   )
@@
   (no_connect (at 339.09 74.93))
   (no_connect (at 339.09 49.53))
+  (no_connect (at 280.67 39.37))
   (no_connect (at 119.38 144.78))
   (no_connect (at 384.81 72.39))
@@
     (stroke (width 0) (type default) (color 0 0 0 0))
   )
-  (wire (pts (xy 283.21 31.75) (xy 283.21 34.29))
-    (stroke (width 0) (type default) (color 0 0 0 0))
-  )
   (wire (pts (xy 27.94 135.89) (xy 30.48 135.89))
     (stroke (width 0) (type default) (color 0 0 0 0))
@@
     (stroke (width 0) (type default) (color 0 0 0 0))
   )
-  (wire (pts (xy 283.21 34.29) (xy 280.67 34.29))
-    (stroke (width 0) (type default) (color 0 0 0 0))
-  )
   (wire (pts (xy 127 19.05) (xy 127 21.59))
     (stroke (width 0) (type default) (color 0 0 0 0))
@@
     (stroke (width 0) (type default) (color 0 0 0 0))
   )
-  (wire (pts (xy 290.83 39.37) (xy 294.64 39.37))
-    (stroke (width 0) (type default) (color 0 0 0 0))
-  )
   (wire (pts (xy 118.11 110.49) (xy 101.6 110.49))
     (stroke (width 0) (type default) (color 0 0 0 0))
@@
     (stroke (width 0) (type default) (color 0 0 0 0))
   )
-  (wire (pts (xy 294.64 31.75) (xy 283.21 31.75))
-    (stroke (width 0) (type default) (color 0 0 0 0))
-  )
   (polyline (pts (xy 182.88 21.59) (xy 309.88 21.59))
     (stroke (width 0) (type default) (color 0 0 0 0))
@@
     (stroke (width 0) (type default) (color 0 0 0 0))
   )
-  (wire (pts (xy 284.48 34.29) (xy 283.21 34.29))
+  (wire (pts (xy 280.67 34.29) (xy 284.48 34.29))
     (stroke (width 0) (type default) (color 0 0 0 0))
   )
@@
     (stroke (width 0) (type default) (color 0 0 0 0))
   )
-  (wire (pts (xy 294.64 39.37) (xy 294.64 31.75))
-    (stroke (width 0) (type default) (color 0 0 0 0))
-  )
   (wire (pts (xy 200.66 88.9) (xy 200.66 99.06))
     (stroke (width 0) (type default) (color 0 0 0 0))
@@
     (effects (font (size 1.27 1.27)) (justify left bottom))
   )
-  (label "uart_mux_tx" (at 48.26 179.07 0)
-    (effects (font (size 1.27 1.27)) (justify left bottom))
-  )
   (label "s8_en_1" (at 224.79 138.43 0)
     (effects (font (size 1.27 1.27)) (justify left bottom))
@@
     (effects (font (size 1.27 1.27)) (justify left bottom))
   )
-  (label "uart_mux_rx" (at 48.26 173.99 0)
-    (effects (font (size 1.27 1.27)) (justify left bottom))
-  )
   (label "sr_clear" (at 384.81 59.69 0)
     (effects (font (size 1.27 1.27)) (justify left bottom))
@@
     (effects (font (size 1.27 1.27)) (justify left bottom))
   )
-  (label "esp_tx" (at 48.26 166.37 0)
-    (effects (font (size 1.27 1.27)) (justify left bottom))
-  )
   (label "s8_out_1" (at 91.44 46.99 0)
     (effects (font (size 1.27 1.27)) (justify left bottom))
@@
     (effects (font (size 1.27 1.27)) (justify right bottom))
   )
-  (label "esp_rx" (at 48.26 161.29 0)
-    (effects (font (size 1.27 1.27)) (justify left bottom))
-  )
   (label "s2_out_1" (at 91.44 31.75 0)
     (effects (font (size 1.27 1.27)) (justify left bottom))
@@
     (pin "1")
   )
-  (symbol (lib_id "Connector:TestPoint") (at 48.26 166.37 90) (unit 1)
-    (in_bom yes) (on_board yes)
-    (property "Reference" "TP2" (id 0) (at 41.91 166.37 90))
-    (property "Value" "TestPoint" (id 1) (at 41.91 165.1 90))
-    (property "Footprint" "TestPoint:TestPoint_Pad_2.0x2.0mm" (id 2) (at 48.26 161.29 0)
-      (effects (font (size 1.27 1.27)) hide)
-    )
-    (property "Datasheet" "~" (id 3) (at 48.26 161.29 0)
-      (effects (font (size 1.27 1.27)) hide)
-    )
-    (pin "1")
-  )
   (symbol (lib_id "power:GND3") (at 46.99 33.02 0) (unit 1)
     (in_bom yes) (on_board yes) (fields_autoplaced)
@@
     (pin "1")
   )
-  (symbol (lib_id "Jumper:Jumper_2_Bridged") (at 285.75 39.37 0) (unit 1)
-    (in_bom yes) (on_board yes)
-    (property "Reference" "JP1" (id 0) (at 292.1 36.83 0))
-    (property "Value" "Jumper_2_Bridged" (id 1) (at 285.75 38.1 0))
-    (property "Footprint" "Jumper:SolderJumper-2_P1.3mm_Open_RoundedPad1.0x1.5mm" (id 2) (at 285.75 39.37 0)
-      (effects (font (size 1.27 1.27)) hide)
-    )
-    (property "Datasheet" "~" (id 3) (at 285.75 39.37 0)
-      (effects (font (size 1.27 1.27)) hide)
-    )
-    (pin "1")
-    (pin "2")
-  )
   (symbol (lib_id "power:GND1") (at 114.3 63.5 0) (unit 1)
     (in_bom yes) (on_board yes)
@@
     (pin "1")
   )
-  (symbol (lib_id "Connector:TestPoint") (at 48.26 161.29 90) (unit 1)
-    (in_bom yes) (on_board yes)
-    (property "Reference" "TP1" (id 0) (at 41.91 161.29 90))
-    (property "Value" "TestPoint" (id 1) (at 41.91 160.02 90))
-    (property "Footprint" "TestPoint:TestPoint_Pad_2.0x2.0mm" (id 2) (at 48.26 156.21 0)
-      (effects (font (size 1.27 1.27)) hide)
-    )
-    (property "Datasheet" "~" (id 3) (at 48.26 156.21 0)
-      (effects (font (size 1.27 1.27)) hide)
-    )
-    (pin "1")
-  )
   (symbol (lib_id "power:GNDA") (at 128.27 81.28 0) (unit 1)
     (in_bom yes) (on_board yes) (fields_autoplaced)
@@
     (pin "1")
   )
-  (symbol (lib_id "Connector:TestPoint") (at 48.26 173.99 90) (unit 1)
-    (in_bom yes) (on_board yes)
-    (property "Reference" "TP3" (id 0) (at 41.91 173.99 90))
-    (property "Value" "TestPoint" (id 1) (at 41.91 172.72 90))
-    (property "Footprint" "TestPoint:TestPoint_Pad_2.0x2.0mm" (id 2) (at 48.26 168.91 0)
-      (effects (font (size 1.27 1.27)) hide)
-    )
-    (property "Datasheet" "~" (id 3) (at 48.26 168.91 0)
-      (effects (font (size 1.27 1.27)) hide)
-    )
-    (pin "1")
-  )
   (symbol (lib_id "power:GND1") (at 217.17 55.88 0) (unit 1)
     (in_bom yes) (on_board yes) (fields_autoplaced)
@@
     (pin "6")
   )
-  (symbol (lib_id "Connector:TestPoint") (at 48.26 179.07 90) (unit 1)
-    (in_bom yes) (on_board yes)
-    (property "Reference" "TP4" (id 0) (at 41.91 179.07 90))
-    (property "Value" "TestPoint" (id 1) (at 41.91 177.8 90))
-    (property "Footprint" "TestPoint:TestPoint_Pad_2.0x2.0mm" (id 2) (at 48.26 173.99 0)
-      (effects (font (size 1.27 1.27)) hide)
-    )
-    (property "Datasheet" "~" (id 3) (at 48.26 173.99 0)
-      (effects (font (size 1.27 1.27)) hide)
-    )
-    (pin "1")
-  )
   (symbol (lib_id "power:GND") (at 24.13 66.04 0) (unit 1)
     (in_bom yes) (on_board yes)
@@
       (reference "J8") (unit 1) (value "Conn_01x02") (footprint "Connector_JST:JST_XA_S02B-XASK-1N-BN_1x02_P2.50mm_Horizontal")
     )
-    (path "/052825ed-e1d2-4641-a08d-515059ea0e67"
-      (reference "JP1") (unit 1) (value "Jumper_2_Bridged") (footprint "Jumper:SolderJumper-2_P1.3mm_Open_RoundedPad1.0x1.5mm")
-    )
     (path "/fa4c15e6-4d31-42fc-b26c-439f4937489e"
       (reference "Q1") (unit 1) (value "AO3400A") (footprint "Package_TO_SOT_SMD:SOT-23")
@@
       (reference "RN5") (unit 1) (value "R_Pack04") (footprint "Resistor_SMD:R_Array_Concave_4x0603")
     )
-    (path "/914564fe-d043-4cfe-932c-53f07fe84a7b"
-      (reference "TP1") (unit 1) (value "TestPoint") (footprint "TestPoint:TestPoint_Pad_2.0x2.0mm")
-    )
-    (path "/01e4ae93-47a4-4529-af0b-5124456e7871"
-      (reference "TP2") (unit 1) (value "TestPoint") (footprint "TestPoint:TestPoint_Pad_2.0x2.0mm")
-    )
-    (path "/f4536eba-1e9f-462c-a2fc-f65fb527354f"
-      (reference "TP3") (unit 1) (value "TestPoint") (footprint "TestPoint:TestPoint_Pad_2.0x2.0mm")
-    )
-    (path "/f7934c4b-083a-4326-ac05-954ce3bc6a74"
-      (reference "TP4") (unit 1) (value "TestPoint") (footprint "TestPoint:TestPoint_Pad_2.0x2.0mm")
-    )
     (path "/00f55aa5-6e34-48cd-b931-6feb0c66bec3"

Commit message: before rearrange
Connections:
- net s10_en_1: now also U10.5 (QF); no longer U10.2 (QC)
- net s11_12_13_en_1: now also U10.7 (QH); no longer U10.15 (QA)
- net s11_out_1: now also U6.5 (AIN1); no longer U6.4 (AIN0)
- net s14_en_1: now also U10.6 (QG); no longer U10.3 (QD)
- net s14_out_1: now also U6.4 (AIN0); no longer U6.5 (AIN1)
- net s1_en_1: now also U8.4 (QE); no longer U8.15 (QA)
- net s5_en_1: now also U8.15 (QA); no longer U8.4 (QE)
- net s6_en_1: now also U8.1 (QB); no longer U8.3 (QD)
- net s8_en_1: now also U8.3 (QD); no longer U8.1 (QB)
- net s9_en_1: now also U10.4 (QE); no longer U10.1 (QB)
- net sr_clear: now also U14.31 (PA6); no longer U14.29 (PA4)
- net sr_latch: now also U14.29 (PA4); no longer U14.31 (PA6)
Changed lines of the file:
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@@
   (no_connect (at 339.09 62.23))
   (no_connect (at 40.64 76.2))
+  (no_connect (at 246.38 161.29))
   (no_connect (at 234.95 55.88))
   (no_connect (at 217.17 43.18))
   (no_connect (at 40.64 57.15))
   (no_connect (at 138.43 100.33))
-  (no_connect (at 246.38 176.53))
+  (no_connect (at 246.38 166.37))
   (no_connect (at 261.62 109.22))
   (no_connect (at 40.64 54.61))
@@
   (no_connect (at 339.09 41.91))
   (no_connect (at 280.67 36.83))
-  (no_connect (at 246.38 173.99))
   (no_connect (at 40.64 52.07))
-  (no_connect (at 246.38 168.91))
   (no_connect (at 384.81 80.01))
   (no_connect (at 339.09 57.15))
@@
   (no_connect (at 384.81 77.47))
   (no_connect (at 297.18 83.82))
+  (no_connect (at 246.38 158.75))
   (no_connect (at 339.09 69.85))
   (no_connect (at 339.09 74.93))
@@
   (no_connect (at 384.81 72.39))
   (no_connect (at 234.95 43.18))
+  (no_connect (at 246.38 163.83))
   (no_connect (at 384.81 46.99))
   (no_connect (at 139.7 137.16))
   (no_connect (at 119.38 147.32))
-  (no_connect (at 246.38 171.45))
   (no_connect (at 234.95 53.34))
   (no_connect (at 246.38 181.61))
@@
     (effects (font (size 1.27 1.27)) (justify left bottom))
   )
+  (label "s8_en_1" (at 224.79 143.51 0)
+    (effects (font (size 1.27 1.27)) (justify left bottom))
+  )
   (label "s9_out_1" (at 91.44 64.77 0)
     (effects (font (size 1.27 1.27)) (justify left bottom))
@@
     (effects (font (size 1.27 1.27)) (justify left bottom))
   )
-  (label "s8_en_1" (at 224.79 138.43 0)
-    (effects (font (size 1.27 1.27)) (justify left bottom))
-  )
   (label "SCL1" (at 87.63 158.75 0)
     (effects (font (size 1.27 1.27)) (justify left bottom))
@@
     (effects (font (size 1.27 1.27)) (justify left bottom))
   )
-  (label "s1_en_1" (at 224.79 135.89 0)
+  (label "s6_en_1" (at 224.79 138.43 0)
     (effects (font (size 1.27 1.27)) (justify left bottom))
   )
@@
     (effects (font (size 1.27 1.27)) (justify left bottom))
   )
+  (label "s5_en_1" (at 224.79 135.89 0)
+    (effects (font (size 1.27 1.27)) (justify left bottom))
+  )
   (label "sr_latch" (at 204.47 148.59 180)
     (effects (font (size 1.27 1.27)) (justify right bottom))
@@
     (effects (font (size 1.27 1.27)) (justify right bottom))
   )
-  (label "s9_en_1" (at 246.38 161.29 0)
-    (effects (font (size 1.27 1.27)) (justify left bottom))
-  )
-  (label "sr_clear" (at 384.81 59.69 0)
-    (effects (font (size 1.27 1.27)) (justify left bottom))
-  )
   (label "particles_tx" (at 288.29 64.77 180)
     (effects (font (size 1.27 1.27)) (justify right bottom))
@@
     (effects (font (size 1.27 1.27)) (justify left bottom))
   )
-  (label "s11_out_1" (at 91.44 52.07 0)
-    (effects (font (size 1.27 1.27)) (justify left bottom))
-  )
   (label "s12_out_1" (at 91.44 59.69 0)
     (effects (font (size 1.27 1.27)) (justify left bottom))
@@
     (effects (font (size 1.27 1.27)) (justify right bottom))
   )
+  (label "sr_clear" (at 384.81 54.61 0)
+    (effects (font (size 1.27 1.27)) (justify left bottom))
+  )
   (label "en_4.2v_signal" (at 339.09 36.83 180)
     (effects (font (size 1.27 1.27)) (justify right bottom))
   )
-  (label "s5_en_1" (at 224.79 146.05 0)
-    (effects (font (size 1.27 1.27)) (justify left bottom))
-  )
   (label "uart_mux_tx" (at 196.85 99.06 180)
     (effects (font (size 1.27 1.27)) (justify right bottom))
@@
     (effects (font (size 1.27 1.27)) (justify left bottom))
   )
-  (label "s10_en_1" (at 246.38 163.83 0)
+  (label "s10_en_1" (at 246.38 171.45 0)
     (effects (font (size 1.27 1.27)) (justify left bottom))
   )
@@
     (effects (font (size 1.27 1.27)) (justify left bottom))
   )
+  (label "sr_latch" (at 384.81 59.69 0)
+    (effects (font (size 1.27 1.27)) (justify left bottom))
+  )
   (label "s14_out_1" (at 86.36 251.46 0)
     (effects (font (size 1.27 1.27)) (justify left bottom))
   )
+  (label "s1_en_1" (at 224.79 146.05 0)
+    (effects (font (size 1.27 1.27)) (justify left bottom))
+  )
   (label "particles_tx" (at 297.18 99.06 0)
     (effects (font (size 1.27 1.27)) (justify left bottom))
@@
     (effects (font (size 1.27 1.27)) (justify left bottom))
   )
+  (label "s11_out_1" (at 91.44 54.61 0)
+    (effects (font (size 1.27 1.27)) (justify left bottom))
+  )
   (label "s8_out_1" (at 86.36 208.28 0)
     (effects (font (size 1.27 1.27)) (justify left bottom))
@@
     (effects (font (size 1.27 1.27)) (justify left bottom))
   )
+  (label "s9_en_1" (at 246.38 168.91 0)
+    (effects (font (size 1.27 1.27)) (justify left bottom))
+  )
   (label "SCL1" (at 339.09 64.77 180)
     (effects (font (size 1.27 1.27)) (justify right bottom))
@@
     (effects (font (size 1.27 1.27)) (justify right bottom))
   )
-  (label "s14_out_1" (at 91.44 54.61 0)
-    (effects (font (size 1.27 1.27)) (justify left bottom))
-  )
   (label "gps_rx" (at 297.18 88.9 0)
     (effects (font (size 1.27 1.27)) (justify left bottom))
@@
     (effects (font (size 1.27 1.27)) (justify right bottom))
   )
-  (label "s14_en_1" (at 246.38 166.37 0)
-    (effects (font (size 1.27 1.27)) (justify left bottom))
-  )
   (label "s10_en_1" (at 86.36 256.54 0)
     (effects (font (size 1.27 1.27)) (justify left bottom))
@@
     (effects (font (size 1.27 1.27)) (justify left bottom))
   )
+  (label "s11_12_13_en_1" (at 246.38 176.53 0)
+    (effects (font (size 1.27 1.27)) (justify left bottom))
+  )
   (label "esp_rx" (at 339.09 44.45 180)
     (effects (font (size 1.27 1.27)) (justify right bottom))
   )
+  (label "s14_out_1" (at 91.44 52.07 0)
+    (effects (font (size 1.27 1.27)) (justify left bottom))
+  )
   (label "s11_out_1" (at 86.36 238.76 0)
     (effects (font (size 1.27 1.27)) (justify left bottom))
@@
     (effects (font (size 1.27 1.27)) (justify right bottom))
   )
-  (label "sr_latch" (at 384.81 54.61 0)
-    (effects (font (size 1.27 1.27)) (justify left bottom))
-  )
   (label "s9_en_1" (at 86.36 259.08 0)
     (effects (font (size 1.27 1.27)) (justify left bottom))
@@
     (effects (font (size 1.27 1.27)) (justify left bottom))
   )
+  (label "s14_en_1" (at 246.38 173.99 0)
+    (effects (font (size 1.27 1.27)) (justify left bottom))
+  )
   (label "s6_out_1" (at 86.36 218.44 0)
     (effects (font (size 1.27 1.27)) (justify left bottom))
   )
-  (label "s6_en_1" (at 224.79 143.51 0)
-    (effects (font (size 1.27 1.27)) (justify left bottom))
-  )
   (label "s13_out_1" (at 86.36 233.68 0)
     (effects (font (size 1.27 1.27)) (justify left bottom))
@@
     (effects (font (size 1.27 1.27)) (justify left bottom))
   )
-  (label "s11_12_13_en_1" (at 246.38 158.75 0)
-    (effects (font (size 1.27 1.27)) (justify left bottom))
-  )

Commit message: in progress
Parts:
- added JP1: Jumper_2_Bridged, Jumper:SolderJumper-2_P1.3mm_Open_TrianglePad1.0x1.5mm, symbol Jumper:Jumper_2_Bridged
- J7, J8: footprint Connector_JST:JST_XA_S02B-XASK-1N-BN_1x02_P2.50mm_Horizontal -> Connector_JST:JST_XA_B02B-XASK-1_1x02_P2.50mm_Vertical
Connections:
- net GND: now also JP1.2 (B); no longer C1.2, C2.2, C3.2, C4.2, J5.1 (Pin_1), J6.2 (Pin_2), U4.1 (ADDR), U4.3 (GND), U5.3 (GND), U6.1 (ADDR), U6.3 (GND), U7.3 (GND)
- net s11_out_1: now also U6.4 (AIN0); no longer U6.5 (AIN1)
- net s14_out_1: no longer U6.4 (AIN0)
- net s1_out_1: now also U4.4 (AIN0); no longer U4.5 (AIN1)
- net s2_out_1: now also U4.5 (AIN1); no longer U4.4 (AIN0)
- new net GND3: C1.2, C2.2, C3.2, C4.2, J5.1 (Pin_1), J6.2 (Pin_2), JP1.1 (A), U4.1 (ADDR), U4.3 (GND), U5.3 (GND), U6.1 (ADDR), U6.3 (GND), U7.3 (GND)
