File: super-met v6/super-met-v6/super-met-v6.kicad_sch (KiCad schematic)
At the start: 55 parts, among them J1 Conn_01x02, J2 Conn_01x08, J3 Conn_01x08, J4 Conn_01x04, J5 Conn_01x08, J6 Conn_01x04, J7 Conn_01x02, J8 Conn_01x02, Q1 AO3400A, Q10 AO3400A, Q11 AO3400A, Q12 AO3400A, Q2 AO3400A, Q3 AO3400A, Q4 AO3400A, Q5 AO3400A, Q6 AO3400A, Q7 AO3400A, Q8 AO3400A, Q9 AO3400A, U1 DC-DC_MOD, U10 74HC595, U11 GY-GPS6MV2, U12 ESP-01v090, U13 74HC4052D, U14 BLUEPILL, U2 DC-DC_MOD, U3 DC-DC_MOD, U4 ADS1115IDGS, U5 ADS1115IDGS, U6 ADS1115IDGS, U7 ADS1115IDGS, U8 74HC595, U9 SIM800L

Commit message: almost done?
Parts:
- removed H3: MountingHole, MountingHole:MountingHole_3.2mm_M3, symbol Mechanical:MountingHole
- added TP1, TP2, TP3, TP4, TP6, TP7, TP8, TP9, TP? (x2): TestPoint, TestPoint:TestPoint_Pad_2.0x2.0mm, symbol Connector:TestPoint
Connections:
- net SCL1: now also TP2.1
- net SCL2: now also TP9.1
- net SDA1: now also TP1.1
- net SDA2: now also TP8.1
- net esp_rx: now also TP?.1
- net esp_tx: now also TP?.1
- net uart_mux_rx: now also TP3.1
- net uart_mux_s0: now also TP7.1
- net uart_mux_s1: now also TP6.1
- net uart_mux_tx: now also TP4.1

Commit message: almost done?
Parts:
- gave numbers to parts that had none: 2
Changed lines of the file:
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@@
   (symbol (lib_id "Connector:TestPoint") (at 26.67 212.09 90) (unit 1)
     (in_bom yes) (on_board yes)
-    (property "Reference" "TP?" (id 0) (at 20.32 212.09 90))
+    (property "Reference" "TP11" (id 0) (at 20.32 212.09 90))
     (property "Value" "TestPoint" (id 1) (at 20.32 210.82 90))
     (property "Footprint" "TestPoint:TestPoint_Pad_2.0x2.0mm" (id 2) (at 26.67 207.01 0)
@@
   (symbol (lib_id "Connector:TestPoint") (at 26.67 208.28 90) (unit 1)
     (in_bom yes) (on_board yes)
-    (property "Reference" "TP?" (id 0) (at 20.32 208.28 90))
+    (property "Reference" "TP10" (id 0) (at 20.32 208.28 90))
     (property "Value" "TestPoint" (id 1) (at 20.32 207.01 90))
     (property "Footprint" "TestPoint:TestPoint_Pad_2.0x2.0mm" (id 2) (at 26.67 203.2 0)
@@
       (reference "TP9") (unit 1) (value "TestPoint") (footprint "TestPoint:TestPoint_Pad_2.0x2.0mm")
     )
+    (path "/fde5fc6a-901e-4eb7-9a63-4921ec72a024"
+      (reference "TP10") (unit 1) (value "TestPoint") (footprint "TestPoint:TestPoint_Pad_2.0x2.0mm")
+    )
     (path "/3ff9388d-99f6-47cc-8d35-6f9369555500"
-      (reference "TP?") (unit 1) (value "TestPoint") (footprint "TestPoint:TestPoint_Pad_2.0x2.0mm")
-    )
-    (path "/fde5fc6a-901e-4eb7-9a63-4921ec72a024"
-      (reference "TP?") (unit 1) (value "TestPoint") (footprint "TestPoint:TestPoint_Pad_2.0x2.0mm")
+      (reference "TP11") (unit 1) (value "TestPoint") (footprint "TestPoint:TestPoint_Pad_2.0x2.0mm")
     )
     (path "/f63ee7d4-ecc1-488b-9f90-733ee9f9aa08"

Commit message: before_changing_fills
Connections:
- net 4.2v: no longer R3.2
- net GND: now also R3.2
Changed lines of the file:
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@@
   (junction (at 227.33 76.2) (diameter 0) (color 0 0 0 0)
   )
+  (junction (at 35.56 85.09) (diameter 0) (color 0 0 0 0)
+  )
   (junction (at 214.63 163.83) (diameter 0) (color 0 0 0 0)
-  )
-  (junction (at 35.56 87.63) (diameter 0) (color 0 0 0 0)
   )
   (junction (at 226.06 99.06) (diameter 0) (color 0 0 0 0)
@@
     (stroke (width 0) (type default) (color 0 0 0 0))
   )
-  (wire (pts (xy 35.56 87.63) (xy 35.56 95.25))
-    (stroke (width 0) (type default) (color 0 0 0 0))
-  )
   (wire (pts (xy 209.55 87.63) (xy 214.63 87.63))
     (stroke (width 0) (type default) (color 0 0 0 0))
@@
     (stroke (width 0) (type default) (color 0 0 0 0))
   )
-  (wire (pts (xy 35.56 87.63) (xy 40.64 87.63))
-    (stroke (width 0) (type default) (color 0 0 0 0))
-  )
   (wire (pts (xy 62.23 27.94) (xy 62.23 33.02))
     (stroke (width 0) (type default) (color 0 0 0 0))
@@
     (stroke (width 0) (type default) (color 0 0 0 0))
   )
-  (wire (pts (xy 31.75 87.63) (xy 35.56 87.63))
+  (wire (pts (xy 31.75 87.63) (xy 40.64 87.63))
     (stroke (width 0) (type default) (color 0 0 0 0))
   )
@@
     (stroke (width 0) (type default) (color 0 0 0 0))
   )
+  (wire (pts (xy 35.56 85.09) (xy 35.56 95.25))
+    (stroke (width 0) (type default) (color 0 0 0 0))
+  )
   (wire (pts (xy 204.47 151.13) (xy 204.47 163.83))
     (stroke (width 0) (type default) (color 0 0 0 0))
@@
     (stroke (width 0) (type default) (color 0 0 0 0))
   )
-  (wire (pts (xy 26.67 85.09) (xy 40.64 85.09))
+  (wire (pts (xy 26.67 85.09) (xy 35.56 85.09))
     (stroke (width 0) (type default) (color 0 0 0 0))
   )
@@
     (stroke (width 0) (type default) (color 0 0 0 0))
   )
+  (wire (pts (xy 35.56 85.09) (xy 40.64 85.09))
+    (stroke (width 0) (type default) (color 0 0 0 0))
+  )
